File: Hardware/kicad/amplituner/amplituner/Ultra kombajn audio.sch (KiCad schematic (older format))
At the start: 129 parts, among them U1 LM3886, U2 LM3886, U3 LM3886, U4 LM3886, U5 STM32L4Q5, U6 TDA7719

Commit message: new
Parts:
- gave numbers to parts that had none: 12
Changed lines of the file:
@@
 Radio
 $Comp
-L Device:Crystal Y?
+L Device:Crystal Y1
 U 1 1 62A22890
 P 9800 1550
-F 0 "Y?" V 9750 1300 50  0000 L CNN
+F 0 "Y1" V 9750 1300 50  0000 L CNN
 F 1 "Crystal" V 9900 1200 50  0000 L CNN
 F 2 "" H 9800 1550 50  0001 C CNN
@@
 $EndComp
 $Comp
-L Device:C C?
+L Device:C C79
 U 1 1 62A24053
 P 9500 1750
-F 0 "C?" V 9350 1650 50  0000 C CNN
+F 0 "C79" V 9350 1650 50  0000 C CNN
 F 1 "C" V 9450 1650 50  0000 C CNN
 F 2 "" H 9538 1600 50  0001 C CNN
@@
 $EndComp
 $Comp
-L Device:C C?
+L Device:C C78
 U 1 1 62A24A2E
 P 9500 1350
-F 0 "C?" V 9650 1250 50  0000 C CNN
+F 0 "C78" V 9650 1250 50  0000 C CNN
 F 1 "C" V 9550 1250 50  0000 C CNN
 F 2 "" H 9538 1200 50  0001 C CNN
@@
 	9300 1350 9350 1350
 $Comp
-L power:GNDD #PWR?
+L power:GNDD #PWR08
 U 1 1 62AB52D7
 P 9300 1550
-F 0 "#PWR?" H 9300 1300 50  0001 C CNN
+F 0 "#PWR08" H 9300 1300 50  0001 C CNN
 F 1 "GNDD" H 9304 1395 50  0000 C CNN
 F 2 "" H 9300 1550 50  0001 C CNN
@@
 Main Power
 $Comp
-L Electronic_stethoscope-cache:Transistor_BJT_BC817 Q?
+L Electronic_stethoscope-cache:Transistor_BJT_BC817 Q1
 U 1 1 62B6F6B2
 P 15800 5950
-F 0 "Q?" H 15990 5996 50  0000 L CNN
+F 0 "Q1" H 15990 5996 50  0000 L CNN
 F 1 "BC817" H 15990 5905 50  0000 L CNN
 F 2 "Package_TO_SOT_SMD:SOT-23" H 16000 5875 50  0001 L CIN
@@
 $EndComp
 $Comp
-L Device:LED D?
+L Device:LED D5
 U 1 1 62B71963
 P 15900 5550
-F 0 "D?" V 15939 5432 50  0000 R CNN
+F 0 "D5" V 15939 5432 50  0000 R CNN
 F 1 "LED" V 15848 5432 50  0000 R CNN
 F 2 "" H 15900 5550 50  0001 C CNN
@@
 $EndComp
 $Comp
-L power:GNDD #PWR?
+L power:GNDD #PWR013
 U 1 1 62B8FC8A
 P 15900 6150
-F 0 "#PWR?" H 15900 5900 50  0001 C CNN
+F 0 "#PWR013" H 15900 5900 50  0001 C CNN
 F 1 "GNDD" H 15904 5995 50  0000 C CNN
 F 2 "" H 15900 6150 50  0001 C CNN
@@
 	15900 5750 15900 5700
 $Comp
-L power:+12V #PWR?
+L power:+12V #PWR012
 U 1 1 62BADC8E
 P 15900 5400
-F 0 "#PWR?" H 15900 5250 50  0001 C CNN
+F 0 "#PWR012" H 15900 5250 50  0001 C CNN
 F 1 "+12V" H 15750 5500 50  0000 C CNN
 F 2 "" H 15900 5400 50  0001 C CNN
@@
 TIM16_CH1
 $Comp
-L Switch:SW_Push SW?
+L Switch:SW_Push SW1
 U 1 1 62C52A34
 P 13950 6000
-F 0 "SW?" H 13950 6285 50  0000 C CNN
+F 0 "SW1" H 13950 6285 50  0000 C CNN
 F 1 "Power Button" H 13950 6194 50  0000 C CNN
 F 2 "" H 13950 6200 50  0001 C CNN
@@
 $EndComp
 $Comp
-L Device:R R?
+L Device:R R30
 U 1 1 62C53C1C
 P 14250 5550
-F 0 "R?" H 14320 5596 50  0000 L CNN
+F 0 "R30" H 14320 5596 50  0000 L CNN
 F 1 "R" H 14320 5505 50  0000 L CNN
 F 2 "" V 14180 5550 50  0001 C CNN
@@
 POWER_BUTTON
 $Comp
-L power:GNDD #PWR?
+L power:GNDD #PWR09
 U 1 1 62C9136A
 P 13950 6200
-F 0 "#PWR?" H 13950 5950 50  0001 C CNN
+F 0 "#PWR09" H 13950 5950 50  0001 C CNN
 F 1 "GNDD" H 13954 6045 50  0000 C CNN
 F 2 "" H 13950 6200 50  0001 C CNN
@@
 $EndComp
 $Comp
-L Electronic_stethoscope-cache:+3.3V #PWR?
+L Electronic_stethoscope-cache:+3.3V #PWR010
 U 1 1 62CAFB94
 P 14250 5400
-F 0 "#PWR?" H 14250 5250 50  0001 C CNN
+F 0 "#PWR010" H 14250 5250 50  0001 C CNN
 F 1 "+3.3V" H 14400 5500 50  0000 C CNN
 F 2 "" H 14250 5400 50  0001 C CNN
@@
 $EndComp
 $Comp
-L Device:C C?
+L Device:C C80
 U 1 1 62D2A5D1
 P 14250 6050
-F 0 "C?" H 14365 6096 50  0000 L CNN
+F 0 "C80" H 14365 6096 50  0000 L CNN
 F 1 "C" H 14365 6005 50  0000 L CNN
 F 2 "" H 14288 5900 50  0001 C CNN
@@
 $EndComp
 $Comp
-L Device:R R?
+L Device:R R29
 U 1 1 62D2B1DB
 P 14100 5800
-F 0 "R?" H 14170 5846 50  0000 L CNN
+F 0 "R29" H 14170 5846 50  0000 L CNN
 F 1 "R" H 14170 5755 50  0000 L CNN
 F 2 "" V 14030 5800 50  0001 C CNN
@@
 	14250 5900 14250 5800
 $Comp
-L power:GNDD #PWR?
+L power:GNDD #PWR011
 U 1 1 62D85255
 P 14250 6200
-F 0 "#PWR?" H 14250 5950 50  0001 C CNN
+F 0 "#PWR011" H 14250 5950 50  0001 C CNN
 F 1 "GNDD" H 14254 6045 50  0000 C CNN
 F 2 "" H 14250 6200 50  0001 C CNN
@@
 Wire Notes Line
 	13500 6450 13500 5050
-Wire Notes Line
-	13500 5050 16400 5050
 Text Notes 13550 5200 0    79   ~ 0
 Power button with LED
@@
 Text Notes 950  13000 0    197  ~ 39
 Blutetooth
-Wire Notes Line
-	13500 5400 11100 5400
-Text Notes 11200 5600 0    79   ~ 0
+Text Notes 10400 5200 0    79   ~ 0
 USB
 Wire Notes Line width 12
@@
 MCU - ESP8266\n
 $Comp
-L ESP8266-12E_ESP-12E:ESP8266-12E_ESP-12E U?
+L ESP8266-12E_ESP-12E:ESP8266-12E_ESP-12E U9
 U 1 1 63075F38
 P 12700 11850
-F 0 "U?" H 12700 12717 50  0000 C CNN
+F 0 "U9" H 12700 12717 50  0000 C CNN
 F 1 "ESP8266-12E_ESP-12E" H 12700 12626 50  0000 C CNN
 F 2 "RF_Module:ESP-12E" H 12700 11850 50  0001 L BNN
@@
 $EndComp
 $Comp
-L Audio:CS43L21 U?
+L Audio:CS43L21 U7
 U 1 1 63079887
 P 7450 13200
-F 0 "U?" H 7450 12211 50  0000 C CNN
+F 0 "U7" H 7450 12211 50  0000 C CNN
 F 1 "CS43L21" H 7450 12120 50  0000 C CNN
 F 2 "Package_DFN_QFN:QFN-32-1EP_5x5mm_P0.5mm_EP3.45x3.45mm" H 7450 13200 50  0001 C CNN
@@
 eeprom
 $Comp
-L Memory_EEPROM:CAT24C256 U?
+L Memory_EEPROM:CAT24C256 U8
 U 1 1 6313C8C5
 P 12300 14950
-F 0 "U?" H 12300 15431 50  0000 C CNN
+F 0 "U8" H 12300 15431 50  0000 C CNN
 F 1 "CAT24C256" H 12300 15340 50  0000 C CNN
 F 2 "" H 12300 14950 50  0001 C CNN
@@
 Wire Notes Line width 12
 	6150 650  16400 650
+Wire Notes Line
+	10350 5050 10350 6450
+Wire Notes Line
+	10350 5050 16400 5050
 $EndSCHEMATC
