File: Hardware/kicad/block diagram/block-sch/block-sch.sch (KiCad schematic (older format))
At the start: 14 parts

Commit message: new
Connections:
- net labels added: GPIOs
- wire segments 120 -> 130
Other:
- note added: "Encoders and buttons"
- moved on the sheet: D?, LS?

Commit message: new
Parts:
- added H1, H2, H3, H4, H5, H6: MountingHole, MountingHole:MountingHole_3mm_Pad_Via, symbol Mechanical:MountingHole
- C1, C2: renamed from C?; footprint (none) -> Capacitor_THT:CP_Radial_D18.0mm_P7.50mm
- D1: renamed from D?; footprint (none) -> Diode_THT:D_DO-201AE_P12.70mm_Horizontal
- D2, D3, D4: renamed from D?; footprint (none) -> Diode_THT:Diode_Bridge_19.0x3.5x10.0mm_P5.0mm
- R1: renamed from R?; footprint (none) -> Resistor_SMD:R_1206_3216Metric
- gave numbers to parts that had none: 7
Connections:
- net labels added: +15V, ADC
- wire segments 130 -> 125
Other:
- note added: "Analog part of calculating FFT\n and uv meter for display"
- note added: "FFT and UV meter"
- note added: "Power amplifier\n4x LM3886"
- note added: "Six encoders for audio control\n(volume front, volume back, bass, \ntreble, middle, loudness).\nOne encoder for radio.\nFour buttons for user"
- note removed: "Power amplifier\n2x LM3886"

Commit message: new
Parts:
- added F1, F2, F3: Fuse, symbol Device:Fuse
Connections:
- wire segments 125 -> 127
Changed lines of the file:
@@
 $EndSheet
 Wire Wire Line
-	5400 1350 6850 1350
+	5400 1350 5900 1350
 Connection ~ 5400 1350
 Wire Wire Line
 	5400 1700 6850 1700
 Wire Wire Line
-	5400 2050 6850 2050
+	5400 2050 5900 2050
 Connection ~ 5400 2050
 Wire Wire Line
@@
 Six encoders for audio control\n(volume front, volume back, bass, \ntreble, middle, loudness).\nOne encoder for radio.\nFour buttons for user
 Wire Wire Line
-	3900 2750 3900 3150
+	3900 2750 3900 2850
 Connection ~ 3900 3150
 $Comp
@@
 Wire Wire Line
 	5250 4750 5250 5600
+$Comp
+L Device:Fuse F2
+U 1 1 61D5BD98
+P 6050 1350
+F 0 "F2" V 6247 1350 50  0000 C CNN
+F 1 "Fuse" V 6156 1350 50  0000 C CNN
+F 2 "" V 5980 1350 50  0001 C CNN
+F 3 "~" H 6050 1350 50  0001 C CNN
+	1    6050 1350
+	0    -1   -1   0
+$EndComp
+Wire Wire Line
+	6200 1350 6850 1350
+$Comp
+L Device:Fuse F3
+U 1 1 61D5C912
+P 6050 2050
+F 0 "F3" V 6247 2050 50  0000 C CNN
+F 1 "Fuse" V 6156 2050 50  0000 C CNN
+F 2 "" V 5980 2050 50  0001 C CNN
+F 3 "~" H 6050 2050 50  0001 C CNN
+	1    6050 2050
+	0    -1   -1   0
+$EndComp
+Wire Wire Line
+	6200 2050 6850 2050
+$Comp
+L Device:Fuse F1
+U 1 1 61D5DB71
+P 3900 3000
+F 0 "F1" H 3750 3000 50  0000 L CNN
+F 1 "Fuse" H 3700 2900 50  0000 L CNN
+F 2 "" V 3830 3000 50  0001 C CNN
+F 3 "~" H 3900 3000 50  0001 C CNN
+	1    3900 3000
+	1    0    0    -1
+$EndComp
 $EndSCHEMATC
