File: Hardware/kicad/block diagram/block-sch/low_power_scheet.sch (KiCad schematic (older format))
At the start: 23 parts, among them U10 AZ1117-3.3, U8 LM7812_TO220, U9 LM78M05_TO252

Commit message: new
Parts:
- added D10: TVS 3,6V, DIOM5436X247N, symbol lib_amplituner:1SMB5914BT3G
- added D11: TVS 6V, DIOM5436X247N, symbol lib_amplituner:1SMB5914BT3G
- added D12: TVS 15V, DIOM5436X247N, symbol lib_amplituner:1SMB5914BT3G
- added R32, R33, R34, R35, R36, R37: R, Resistor_SMD:R_1206_3216Metric, symbol Device:R
- D13, D14, D15: renamed from D?; footprint (none) -> LED_SMD:LED_1206_3216Metric
- R38, R39, R40: renamed from R?; footprint (none) -> Resistor_SMD:R_1206_3216Metric
Connections:
- net +12V: now also D12.C
- net +15V: now also R32.1, R33.1, R34.1, R35.1, R36.1, R37.1; no longer C83.1, C84.1, C85.1, C86.1, C87.1, C88.1, U10.3 (VI), U8.1 (VI), U9.1 (VI)
- net +5V: now also D11.C
- net GNDA: now also D12.A
- net GNDD: now also C85.1, C88.1, U10.3 (VI), D10.A, D10.C, D11.A, R33.2, R36.2
- new net: C84.1, C87.1, R32.2, R35.2, U9.1 (VI)
- new net: C83.1, C86.1, R34.2, R37.2, U8.1 (VI)
Other:
- moved on the sheet: C85, C88, C89, C90, C91, C93, C94, C95, C96, C97, D13, D14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
