File: Hardware/kicad/block diagram/block-sch/stm32_scheet.sch (KiCad schematic (older format))
At the start: 14 parts, among them Q2 BC817, SW1 Power Button, U6 STM32L4Q5, Y1 Crystal

Commit message: new
Parts:
- added C92, C98: C, Capacitor_SMD:C_1206_3216Metric, symbol Device:C
- added L1, L2: L, Inductor_SMD:L_1206_3216Metric, symbol Device:L
Connections:
- net +3V3: now also C92.2, L2.1
- net GNDD: now also C92.1, C98.1, L1.2
- net at U6.12 (VSSA): now also L1.1
- net VDDA: now reaches U6.13 (VDDA)
- net VDDA: now also C98.2, L2.2
Other:
- moved on the sheet: C80, C81, Y1
Changed lines of the file:
@@
 L Device:Crystal Y1
 U 1 1 62A22890
-P 4150 1500
-F 0 "Y1" V 4100 1250 50  0000 L CNN
-F 1 "Crystal" V 4250 1150 50  0000 L CNN
-F 2 "Crystal:Crystal_HC52-6mm_Vertical" H 4150 1500 50  0001 C CNN
-F 3 "~" H 4150 1500 50  0001 C CNN
-	1    4150 1500
+P 5650 1450
+F 0 "Y1" V 5600 1200 50  0000 L CNN
+F 1 "Crystal" V 5750 1100 50  0000 L CNN
+F 2 "Crystal:Crystal_HC52-6mm_Vertical" H 5650 1450 50  0001 C CNN
+F 3 "~" H 5650 1450 50  0001 C CNN
+	1    5650 1450
 	0    -1   -1   0
 $EndComp
@@
 L Device:C C81
 U 1 1 62A24053
-P 3850 1700
-F 0 "C81" V 3700 1600 50  0000 C CNN
-F 1 "C" V 3800 1600 50  0000 C CNN
-F 2 "Capacitor_SMD:C_1206_3216Metric" H 3888 1550 50  0001 C CNN
-F 3 "~" H 3850 1700 50  0001 C CNN
-	1    3850 1700
+P 5350 1650
+F 0 "C81" V 5200 1550 50  0000 C CNN
+F 1 "C" V 5300 1550 50  0000 C CNN
+F 2 "Capacitor_SMD:C_1206_3216Metric" H 5388 1500 50  0001 C CNN
+F 3 "~" H 5350 1650 50  0001 C CNN
+	1    5350 1650
 	0    -1   -1   0
 $EndComp
@@
 L Device:C C80
 U 1 1 62A24A2E
-P 3850 1300
-F 0 "C80" V 4000 1200 50  0000 C CNN
-F 1 "C" V 3900 1200 50  0000 C CNN
-F 2 "Capacitor_SMD:C_1206_3216Metric" H 3888 1150 50  0001 C CNN
-F 3 "~" H 3850 1300 50  0001 C CNN
-	1    3850 1300
-	0    -1   -1   0
-$EndComp
-Wire Wire Line
-	4000 1700 4150 1700
-Wire Wire Line
-	4150 1700 4150 1650
-Wire Wire Line
-	4000 1300 4150 1300
-Wire Wire Line
-	4150 1300 4150 1350
-Wire Wire Line
-	3700 1700 3650 1700
-Wire Wire Line
-	3650 1700 3650 1500
-Wire Wire Line
-	3650 1300 3700 1300
+P 5350 1250
+F 0 "C80" V 5500 1150 50  0000 C CNN
+F 1 "C" V 5400 1150 50  0000 C CNN
+F 2 "Capacitor_SMD:C_1206_3216Metric" H 5388 1100 50  0001 C CNN
+F 3 "~" H 5350 1250 50  0001 C CNN
+	1    5350 1250
+	0    -1   -1   0
+$EndComp
+Wire Wire Line
+	5500 1650 5650 1650
+Wire Wire Line
+	5650 1650 5650 1600
+Wire Wire Line
+	5500 1250 5650 1250
+Wire Wire Line
+	5650 1250 5650 1300
+Wire Wire Line
+	5200 1650 5150 1650
+Wire Wire Line
+	5150 1650 5150 1450
+Wire Wire Line
+	5150 1250 5200 1250
 $Comp
 L power:GNDD #PWR016
 U 1 1 62AB52D7
-P 3650 1500
-F 0 "#PWR016" H 3650 1250 50  0001 C CNN
-F 1 "GNDD" H 3654 1345 50  0000 C CNN
-F 2 "" H 3650 1500 50  0001 C CNN
-F 3 "" H 3650 1500 50  0001 C CNN
-	1    3650 1500
+P 5150 1450
+F 0 "#PWR016" H 5150 1200 50  0001 C CNN
+F 1 "GNDD" H 5154 1295 50  0000 C CNN
+F 2 "" H 5150 1450 50  0001 C CNN
+F 3 "" H 5150 1450 50  0001 C CNN
+	1    5150 1450
 	0    1    1    0
 $EndComp
-Connection ~ 3650 1500
-Wire Wire Line
-	3650 1500 3650 1300
-Text GLabel 4300 1300 2    50   Input ~ 0
+Connection ~ 5150 1450
+Wire Wire Line
+	5150 1450 5150 1250
+Text GLabel 5800 1250 2    50   Input ~ 0
 OSC_IN
-Text GLabel 4300 1700 2    50   Input ~ 0
+Text GLabel 5800 1650 2    50   Input ~ 0
 OSC_OUT
 Wire Wire Line
-	4150 1300 4300 1300
-Connection ~ 4150 1300
-Wire Wire Line
-	4150 1700 4300 1700
-Connection ~ 4150 1700
+	5650 1250 5800 1250
+Connection ~ 5650 1250
+Wire Wire Line
+	5650 1650 5800 1650
+Connection ~ 5650 1650
 $Comp
 L Electronic_stethoscope-cache:Transistor_BJT_BC817 Q2
@@
 Wire Notes Line
 	5150 5150 11200 5150
+$Comp
+L Device:C C92
+U 1 1 61D0C60F
+P 3600 1550
+F 0 "C92" V 3450 1450 50  0000 C CNN
+F 1 "C" V 3550 1450 50  0000 C CNN
+F 2 "Capacitor_SMD:C_1206_3216Metric" H 3638 1400 50  0001 C CNN
+F 3 "~" H 3600 1550 50  0001 C CNN
+	1    3600 1550
+	-1   0    0    1
+$EndComp
+$Comp
+L Device:C C98
+U 1 1 61D0D3C8
+P 4300 1550
+F 0 "C98" V 4150 1450 50  0000 C CNN
+F 1 "C" V 4250 1450 50  0000 C CNN
+F 2 "Capacitor_SMD:C_1206_3216Metric" H 4338 1400 50  0001 C CNN
+F 3 "~" H 4300 1550 50  0001 C CNN
+	1    4300 1550
+	-1   0    0    1
+$EndComp
+$Comp
+L Electronic_stethoscope-cache:+3.3V #PWR030
+U 1 1 61D0D9B2
+P 3600 1200
+F 0 "#PWR030" H 3600 1050 50  0001 C CNN
+F 1 "+3.3V" H 3615 1373 50  0000 C CNN
+F 2 "" H 3600 1200 50  0001 C CNN
+F 3 "" H 3600 1200 50  0001 C CNN
+	1    3600 1200
+	1    0    0    -1
+$EndComp
+$Comp
+L power:GNDD #PWR033
+U 1 1 61D0DFA2
+P 4000 1750
+F 0 "#PWR033" H 4000 1500 50  0001 C CNN
+F 1 "GNDD" H 4004 1595 50  0000 C CNN
+F 2 "" H 4000 1750 50  0001 C CNN
+F 3 "" H 4000 1750 50  0001 C CNN
+	1    4000 1750
+	1    0    0    -1
+$EndComp
+Wire Wire Line
+	3600 1700 4000 1700
+Wire Wire Line
+	4000 1750 4000 1700
+Connection ~ 4000 1700
+Wire Wire Line
+	4000 1700 4300 1700
+Wire Wire Line
+	3600 1400 3600 1300
+Wire Wire Line
+	4300 1400 4300 1300
+Wire Wire Line
+	4300 1300 4100 1300
+Connection ~ 3600 1300
+Wire Wire Line
+	3600 1300 3600 1200
+Text GLabel 2550 2300 2    50   Input ~ 0
+VDDA
+Text GLabel 4300 1300 2    50   Input ~ 0
+VDDA
+$Comp
+L Device:L L2
+U 1 1 61D14F33
+P 3950 1300
+F 0 "L2" V 4140 1300 50  0000 C CNN
+F 1 "L" V 4049 1300 50  0000 C CNN
+F 2 "Inductor_SMD:L_1206_3216Metric" H 3950 1300 50  0001 C CNN
+F 3 "~" H 3950 1300 50  0001 C CNN
+	1    3950 1300
+	0    -1   -1   0
+$EndComp
+Wire Wire Line
+	3800 1300 3600 1300
+$Comp
+L Device:L L1
+U 1 1 61D160ED
+P 2350 6100
+F 0 "L1" H 2403 6146 50  0000 L CNN
+F 1 "L" H 2403 6055 50  0000 L CNN
+F 2 "Inductor_SMD:L_1206_3216Metric" H 2350 6100 50  0001 C CNN
+F 3 "~" H 2350 6100 50  0001 C CNN
+	1    2350 6100
+	1    0    0    -1
+$EndComp
+Wire Wire Line
+	2350 6250 2250 6250
+Wire Wire Line
+	2250 6250 2250 6050
+Connection ~ 2250 6050
+Wire Wire Line
+	2550 2300 2350 2300
+Wire Wire Line
+	2350 2300 2350 2350
 $EndSCHEMATC
