File: Hardware/kicad/block diagram/block-sch/radio_blue.kicad_sch (KiCad schematic)
At the start: 7 parts, among them U11 RDA5807M

Commit message: new
Parts:
- added C105: 100nF, Capacitor_SMD:C_1206_3216Metric, symbol Device:C
- added U12: bluetooth_module, amplituner_lib:bluetooth_module, symbol amplituner_lib_sym:bluetooth_module
Connections:
- net GNDD: now also C105.2, U12.8 (GND)
- net Radio_in_L renamed Radio_L
- net Radio_in_R renamed Radio_R
- new net +5V: C105.1, U12.7 (Vbat)
- new net Bluetooth_IN_G: U12.11 (Lout)
- new net Bluetooth_IN_L: U12.13 (R_out)
- new net Bluetooth_IN_R: U12.12 (Gnd_audio)
- new net NEXT_Butt: U12.3 (NEXT)
- new net PREV_Butt: U12.4 (PREV)
- new net Pause/play_Butt: U12.5 (Pause/play)
Changed lines of the file:
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@@
+    (stroke (width 0) (type default) (color 0 0 0 0))
+  )
+  (wire (pts (xy 121.92 117.602) (xy 125.603 117.602))
+    (stroke (width 0) (type default) (color 0 0 0 0))
+  )
+  (wire (pts (xy 153.543 116.332) (xy 155.956 116.332))
+    (stroke (width 0) (type default) (color 0 0 0 0))
+  )
+  (wire (pts (xy 125.603 134.112) (xy 122.936 134.112))
+    (stroke (width 0) (type default) (color 0 0 0 0))
+  )
+  (wire (pts (xy 153.543 118.872) (xy 155.956 118.872))
+    (stroke (width 0) (type default) (color 0 0 0 0))
+  )
+  (wire (pts (xy 122.174 122.682) (xy 125.603 122.682))
     (stroke (width 0) (type default) (color 0 0 0 0))
   )
@@
     (stroke (width 0) (type default) (color 0 0 0 0))
   )
+  (wire (pts (xy 122.174 120.142) (xy 125.603 120.142))
+    (stroke (width 0) (type default) (color 0 0 0 0))
+  )
   (wire (pts (xy 151.13 69.85) (xy 165.1 69.85))
     (stroke (width 0) (type default) (color 0 0 0 0))
@@
     (stroke (width 0) (type default) (color 0 0 0 0))
   )
+  (wire (pts (xy 122.936 138.43) (xy 113.792 138.43))
+    (stroke (width 0) (type default) (color 0 0 0 0))
+  )
   (wire (pts (xy 119.38 57.15) (xy 107.95 57.15))
     (stroke (width 0) (type default) (color 0 0 0 0))
   )
+  (wire (pts (xy 122.936 131.572) (xy 125.603 131.572))
+    (stroke (width 0) (type default) (color 0 0 0 0))
+  )
   (wire (pts (xy 130.81 59.69) (xy 130.81 57.15))
     (stroke (width 0) (type default) (color 0 0 0 0))
@@
     (stroke (width 0) (type default) (color 0 0 0 0))
   )
+  (wire (pts (xy 153.543 113.792) (xy 156.083 113.792))
+    (stroke (width 0) (type default) (color 0 0 0 0))
+  )
+  (wire (pts (xy 122.936 134.112) (xy 122.936 138.43))
+    (stroke (width 0) (type default) (color 0 0 0 0))
+  )
   (wire (pts (xy 119.38 64.77) (xy 130.81 64.77))
     (stroke (width 0) (type default) (color 0 0 0 0))
   )
+  (wire (pts (xy 122.936 130.81) (xy 122.936 131.572))
+    (stroke (width 0) (type default) (color 0 0 0 0))
+  )
+  (wire (pts (xy 113.792 130.81) (xy 122.936 130.81))
+    (stroke (width 0) (type default) (color 0 0 0 0))
+  )
   (wire (pts (xy 107.95 64.77) (xy 119.38 64.77))
     (stroke (width 0) (type default) (color 0 0 0 0))
+  )
+  (global_label "PREV_Butt" (shape input) (at 122.174 120.142 180) (fields_autoplaced)
+    (effects (font (size 0.9906 0.9906)) (justify right))
+    (property "Intersheet References" "${INTERSHEET_REFS}" (id 0) (at 112.861 120.0801 0)
+      (effects (font (size 0.9906 0.9906)) (justify right) hide)
+    )
+  )
+  (global_label "Pause{slash}play_Butt" (shape input) (at 122.174 122.682 180) (fields_autoplaced)
+    (effects (font (size 0.9906 0.9906)) (justify right))
+    (property "Intersheet References" "${INTERSHEET_REFS}" (id 0) (at 108.0496 122.6201 0)
+      (effects (font (size 0.9906 0.9906)) (justify right) hide)
+    )
+  )
+  (global_label "NEXT_Butt" (shape input) (at 121.92 117.602 180) (fields_autoplaced)
+    (effects (font (size 0.9906 0.9906)) (justify right))
+    (property "Intersheet References" "${INTERSHEET_REFS}" (id 0) (at 112.7014 117.5401 0)
+      (effects (font (size 0.9906 0.9906)) (justify right) hide)
+    )
+  )
+  (global_label "Bluetooth_IN_R" (shape input) (at 155.956 116.332 0) (fields_autoplaced)
+    (effects (font (size 1.27 1.27)) (justify left))
+    (property "Intersheet References" "${INTERSHEET_REFS}" (id 0) (at 265.176 196.342 0)
+      (effects (font (size 1.27 1.27)) hide)
+    )
   )
   (global_label "I2C_SDA" (shape input) (at 130.81 49.53 180) (fields_autoplaced)
@@
     )
   )
-  (global_label "Radio_in_R" (shape input) (at 180.34 69.85 0) (fields_autoplaced)
+  (global_label "Bluetooth_IN_L" (shape input) (at 155.956 118.872 0) (fields_autoplaced)
+    (effects (font (size 1.27 1.27)) (justify left))
+    (property "Intersheet References" "${INTERSHEET_REFS}" (id 0) (at 265.176 195.072 0)
+      (effects (font (size 1.27 1.27)) hide)
+    )
+  )
+  (global_label "Radio_R" (shape input) (at 180.34 69.85 0) (fields_autoplaced)
     (effects (font (size 0.9906 0.9906)) (justify left))
-    (property "Intersheet References" "${INTERSHEET_REFS}" (id 0) (at 0 0 0)
-      (effects (font (size 1.27 1.27)) hide)
-    )
-  )
-  (global_label "Radio_in_L" (shape input) (at 180.34 59.69 0) (fields_autoplaced)
+    (property "Intersheet References" "${INTERSHEET_REFS}" (id 0) (at 188.0491 69.7881 0)
+      (effects (font (size 0.9906 0.9906)) (justify left) hide)
+    )
+  )
+  (global_label "Radio_L" (shape input) (at 180.34 59.69 0) (fields_autoplaced)
     (effects (font (size 0.9906 0.9906)) (justify left))
-    (property "Intersheet References" "${INTERSHEET_REFS}" (id 0) (at 0 0 0)
-      (effects (font (size 1.27 1.27)) hide)
+    (property "Intersheet References" "${INTERSHEET_REFS}" (id 0) (at 187.8604 59.6281 0)
+      (effects (font (size 0.9906 0.9906)) (justify left) hide)
     )
   )
@@
     (effects (font (size 0.9906 0.9906)) (justify left))
     (property "Intersheet References" "${INTERSHEET_REFS}" (id 0) (at 0 0 0)
+      (effects (font (size 1.27 1.27)) hide)
+    )
+  )
+  (global_label "Bluetooth_IN_G" (shape input) (at 156.083 113.792 0) (fields_autoplaced)
+    (effects (font (size 1.27 1.27)) (justify left))
+    (property "Intersheet References" "${INTERSHEET_REFS}" (id 0) (at 265.303 197.612 0)
       (effects (font (size 1.27 1.27)) hide)
     )
@@
     (pin "1")
   )
+  (symbol (lib_id "power:GNDD") (at 113.792 138.43 0) (unit 1)
+    (in_bom yes) (on_board yes)
+    (property "Reference" "#PWR040" (id 0) (at 113.792 144.78 0)
+      (effects (font (size 1.27 1.27)) hide)
+    )
+    (property "Value" "GNDD" (id 1) (at 113.792 142.24 0))
+    (property "Footprint" "" (id 2) (at 113.792 138.43 0)
+      (effects (font (size 1.27 1.27)) hide)
+    )
+    (property "Datasheet" "" (id 3) (at 113.792 138.43 0)
+      (effects (font (size 1.27 1.27)) hide)
+    )
+    (pin "1")
+  )
+  (symbol (lib_id "power:+5V") (at 113.792 130.81 0) (unit 1)
+    (in_bom yes) (on_board yes)
+    (property "Reference" "#PWR04" (id 0) (at 113.792 134.62 0)
+      (effects (font (size 1.27 1.27)) hide)
+    )
+    (property "Value" "+5V" (id 1) (at 113.538 127.254 0))
+    (property "Footprint" "" (id 2) (at 113.792 130.81 0)
+      (effects (font (size 1.27 1.27)) hide)
+    )
+    (property "Datasheet" "" (id 3) (at 113.792 130.81 0)
+      (effects (font (size 1.27 1.27)) hide)
+    )
+    (pin "1")
+  )
+  (symbol (lib_id "amplituner_lib_sym:bluetooth_module") (at 138.303 122.682 0) (unit 1)
+    (in_bom yes) (on_board yes) (fields_autoplaced)
+    (property "Reference" "U12" (id 0) (at 139.573 106.68 0))
+    (property "Value" "bluetooth_module" (id 1) (at 139.573 109.22 0))
+    (property "Footprint" "amplituner_lib:bluetooth_module" (id 2) (at 138.303 122.682 0)
+      (effects (font (size 1.27 1.27)) hide)
+    )
+    (property "Datasheet" "" (id 3) (at 138.303 122.682 0)
+      (effects (font (size 1.27 1.27)) hide)
+    )
+    (pin "1")
+    (pin "10")
+    (pin "11")
+    (pin "12")
+    (pin "13")
+    (pin "14")
+    (pin "19")
+    (pin "2")
+    (pin "20")
+    (pin "3")
+    (pin "4")
+    (pin "5")
+    (pin "6")
+    (pin "7")
+    (pin "8")
+    (pin "9")
+  )
+  (symbol (lib_id "Device:C") (at 113.792 134.62 0) (unit 1)
+    (in_bom yes) (on_board yes)
+    (property "Reference" "C105" (id 0) (at 116.713 133.4516 0)
+      (effects (font (size 1.27 1.27)) (justify left))
+    )
+    (property "Value" "100nF" (id 1) (at 116.713 135.763 0)
+      (effects (font (size 1.27 1.27)) (justify left))
+    )
+    (property "Footprint" "Capacitor_SMD:C_1206_3216Metric" (id 2) (at 114.7572 138.43 0)
+      (effects (font (size 1.27 1.27)) hide)
+    )
+    (property "Datasheet" "~" (id 3) (at 113.792 134.62 0)
+      (effects (font (size 1.27 1.27)) hide)
+    )
+    (pin "1")
+    (pin "2")
+  )
 )
