File: Hardware/kicad/block diagram/block-sch/block-sch.kicad_pcb (KiCad board)
At the start: 2 copper layers, 250 x 100 mm, 140 parts, among them K1 AZ850-x, Q1 BC817, Q2 BC817, U1 LM3886, U2 LM3886, U3 LM3886, U4 LM3886, U5 TDA7719, U6 STM32L4Q5, U7 ESP8266-12E_ESP-12E, Y1 Crystal

Commit message: new
Parts:
- added C100: 100pF, Capacitor_SMD:C_1206_3216Metric, F.Cu at (193.2, 103.7)
- added C101: 10uF, Capacitor_SMD:C_1206_3216Metric, F.Cu at (185.3, 114.8)
- added C102: 10uF, Capacitor_SMD:C_1206_3216Metric, F.Cu at (179.7, 114.8)
- added C83: 100uF Ele, Capacitor_SMD:CP_Elec_4x3.9, F.Cu at (32.5, 142.5)
- added C84: 47uF Tan, lib-amplituner:CAP_TANT_1206_SMD, F.Cu at (40.1, 141.3)
- added C85: 47uF Tan, lib-amplituner:CAP_TANT_1206_SMD, F.Cu at (51.6, 135.5)
- added C86: 100nF, Capacitor_SMD:C_1206_3216Metric, F.Cu at (60.7, 127.2)
- added C87: 100nF, Capacitor_SMD:C_1206_3216Metric, F.Cu at (46.1, 141.3)
- added C88: 100nF, Capacitor_SMD:C_1206_3216Metric, F.Cu at (57.6, 133.9)
- added C89: 100nF, Capacitor_SMD:C_1206_3216Metric, F.Cu at (66.4, 127.2)
- added C90: 100nF, Capacitor_SMD:C_1206_3216Metric, F.Cu at (44.9, 144.7)
- added C91: 100nF, Capacitor_SMD:C_1206_3216Metric, F.Cu at (51.7, 138.8)
- added C92: C, Capacitor_SMD:C_1206_3216Metric, F.Cu at (87.5, 127.2)
- added C93: 47uF Tan, lib-amplituner:CAP_TANT_1206_SMD, F.Cu at (32.3, 147.1)
- added C94: 47uF Tan, lib-amplituner:CAP_TANT_1206_SMD, F.Cu at (54.7, 127.2)
- added C95: 10uF Ele, Capacitor_SMD:CP_Elec_4x3.9, F.Cu at (44.0, 136.7)
- added C96: 100pF, Capacitor_SMD:C_1206_3216Metric, F.Cu at (39.2, 144.7)
- added C97: 100pF, Capacitor_SMD:C_1206_3216Metric, F.Cu at (53.8, 130.6)
- added C98: C, Capacitor_SMD:C_1206_3216Metric, F.Cu at (81.9, 130.6)
- added C99: 100nF, Capacitor_SMD:C_1206_3216Metric, F.Cu at (187.5, 107.2)
- added D13: LED, LED_SMD:LED_1206_3216Metric, F.Cu at (63.3, 130.6)
- added D14: LED, LED_SMD:LED_1206_3216Metric, F.Cu at (51.8, 142.2)
- added D15: LED, LED_SMD:LED_1206_3216Metric, F.Cu at (57.7, 137.3)
- added D9: LED, LED_SMD:LED_1206_3216Metric, F.Cu at (81.9, 127.3)
- added L1: L, Inductor_SMD:L_1206_3216Metric, F.Cu at (76.2, 127.3)
- added L2: L, Inductor_SMD:L_1206_3216Metric, F.Cu at (76.2, 130.7)
- added L3: 100MHz, Inductor_SMD:L_1206_3216Metric, F.Cu at (187.5, 103.8)
- added L4: 100MHz, Inductor_SMD:L_1206_3216Metric, F.Cu at (174.0, 114.9)
- added R32: R, Resistor_SMD:R_1206_3216Metric, F.Cu at (63.0, 143.9)
- added R33: R, Resistor_SMD:R_1206_3216Metric, F.Cu at (56.1, 147.2)
- added R34: R, Resistor_SMD:R_1206_3216Metric, F.Cu at (63.0, 140.6)
- added R35: R, Resistor_SMD:R_1206_3216Metric, F.Cu at (61.7, 147.2)
- added R36: R, Resistor_SMD:R_1206_3216Metric, F.Cu at (57.4, 143.9)
- added R37: R, Resistor_SMD:R_1206_3216Metric, F.Cu at (63.3, 137.2)
- added R38: R, Resistor_SMD:R_1206_3216Metric, F.Cu at (57.4, 140.6)
- added R39: R, Resistor_SMD:R_1206_3216Metric, F.Cu at (50.5, 145.5)
- added R40: R, Resistor_SMD:R_1206_3216Metric, F.Cu at (63.3, 133.9)
- added U10: AZ1117-3.3, lib-amplituner:AZ1117-3.3, F.Cu at (46.2, 129.7)
- added U11: RDA5807M, lib-amplituner:RDA5807M, F.Cu at (177.9, 107.6)
- added U8: LM7812_TO220, Package_TO_SOT_THT:TO-220-3_Vertical, F.Cu at (31.9, 137.5)
- added U9: LM78M05_TO252, Package_TO_SOT_SMD:TO-252-2, F.Cu at (34.7, 129.6)
- moved C2 48.6 mm to (87.5, 100.0)
- moved C1 40.1 mm to (52.5, 102.5)
- moved U5 11.2 mm to (205.0, 130.0)
- moved U6 11.2 mm to (170.0, 130.0)
- moved Y1 11.2 mm to (155.0, 133.8)
- moved D2 9.01 mm to (20.0, 77.5)
- moved D3 9.01 mm to (20.0, 82.5)
- moved D4 9.01 mm to (20.0, 87.5)
- moved U7 5.00 mm to (240.0, 145.0)
Connections:
- net /+36V renamed Net-(C2-Pad2)
- net /-36V renamed Net-(C1-Pad1)
- D2 pad 1: /16V -> +15V
- U6 pad 13: Net-(U6-Pad13) -> VDDA

Commit message: new
Parts:
- moved D5 305.0 mm to (52.1, 108.0)
- moved C75 296.5 mm to (139.7, 130.8), turned to 90 degrees
- moved C63 292.1 mm to (156.2, 141.0), turned to 90 degrees
- moved C70 289.3 mm to (158.8, 141.0), turned to 90 degrees
- moved C74 287.9 mm to (139.7, 134.6)
- moved C64 285.3 mm to (161.3, 141.0), turned to 90 degrees
- moved R8 283.3 mm to (54.6, 96.5)
- moved C26 278.0 mm to (45.7, 73.7)
- moved C15 273.1 mm to (55.9, 116.8)
- moved C73 271.9 mm to (147.3, 125.7)
- moved C16 268.6 mm to (29.2, 104.1)
- moved C7 266.5 mm to (47.0, 108.0)
- moved C27 265.6 mm to (48.3, 85.1)
- moved R24 247.2 mm to (181.6, 108.0)
- moved R14 242.0 mm to (234.9, 106.7)
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Connections:
- K1 pad 2: Net-(K1-Pad2) -> unconnected-(K1-Pad2)
- K1 pad 9: Net-(K1-Pad9) -> unconnected-(K1-Pad9)
- U1 pad 11: Net-(U1-Pad11) -> unconnected-(U1-Pad11)
- U1 pad 2: Net-(U1-Pad2) -> unconnected-(U1-Pad2)
- U1 pad 6: Net-(U1-Pad6) -> unconnected-(U1-Pad6)
- U2 pad 11: Net-(U2-Pad11) -> unconnected-(U2-Pad11)
- U2 pad 2: Net-(U2-Pad2) -> unconnected-(U2-Pad2)
- U2 pad 6: Net-(U2-Pad6) -> unconnected-(U2-Pad6)
- U3 pad 11: Net-(U3-Pad11) -> unconnected-(U3-Pad11)
- U3 pad 2: Net-(U3-Pad2) -> unconnected-(U3-Pad2)
- U3 pad 6: Net-(U3-Pad6) -> unconnected-(U3-Pad6)
- U4 pad 11: Net-(U4-Pad11) -> unconnected-(U4-Pad11)
- U4 pad 2: Net-(U4-Pad2) -> unconnected-(U4-Pad2)
- U4 pad 6: Net-(U4-Pad6) -> unconnected-(U4-Pad6)
- U5 pad 16: Net-(U5-Pad16) -> unconnected-(U5-Pad16)
- U5 pad 17: Net-(U5-Pad17) -> unconnected-(U5-Pad17)
- U5 pad 23: Net-(U5-Pad23) -> unconnected-(U5-Pad23)
- U5 pad 27: Net-(U5-Pad27) -> unconnected-(U5-Pad27)
- U5 pad 28: Net-(U5-Pad28) -> unconnected-(U5-Pad28)
- U6 pad 1: Net-(U6-Pad1) -> unconnected-(U6-Pad1)
- U6 pad 11: Net-(U6-Pad11) -> unconnected-(U6-Pad11)
- U6 pad 2: Net-(U6-Pad2) -> unconnected-(U6-Pad2)
- U6 pad 35: Net-(U6-Pad35) -> unconnected-(U6-Pad35)
- U6 pad 40: Net-(U6-Pad40) -> unconnected-(U6-Pad40)
- U6 pad 43: Net-(U6-Pad43) -> unconnected-(U6-Pad43)
- U6 pad 44: Net-(U6-Pad44) -> unconnected-(U6-Pad44)
- U6 pad 45: Net-(U6-Pad45) -> unconnected-(U6-Pad45)
- U6 pad 52: Net-(U6-Pad52) -> unconnected-(U6-Pad52)
- U6 pad 54: Net-(U6-Pad54) -> unconnected-(U6-Pad54)
- U6 pad 61: Net-(U6-Pad61) -> unconnected-(U6-Pad61)
- U6 pad 62: Net-(U6-Pad62) -> unconnected-(U6-Pad62)
- U6 pad 8: Net-(U6-Pad8) -> unconnected-(U6-Pad8)
- U6 pad 9: Net-(U6-Pad9) -> unconnected-(U6-Pad9)
- U7 pad 1: Net-(U7-Pad1) -> unconnected-(U7-Pad1)
- U7 pad 10: Net-(U7-Pad10) -> unconnected-(U7-Pad10)
- U7 pad 11: Net-(U7-Pad11) -> unconnected-(U7-Pad11)
- U7 pad 12: Net-(U7-Pad12) -> unconnected-(U7-Pad12)
- U7 pad 13: Net-(U7-Pad13) -> unconnected-(U7-Pad13)
- U7 pad 14: Net-(U7-Pad14) -> unconnected-(U7-Pad14)
- U7 pad 15: Net-(U7-Pad15) -> unconnected-(U7-Pad15)
- U7 pad 16: Net-(U7-Pad16) -> unconnected-(U7-Pad16)
- U7 pad 17: Net-(U7-Pad17) -> unconnected-(U7-Pad17)
- U7 pad 18: Net-(U7-Pad18) -> unconnected-(U7-Pad18)
- U7 pad 19: Net-(U7-Pad19) -> unconnected-(U7-Pad19)
- U7 pad 2: Net-(U7-Pad2) -> unconnected-(U7-Pad2)
- U7 pad 20: Net-(U7-Pad20) -> unconnected-(U7-Pad20)
- U7 pad 21: Net-(U7-Pad21) -> unconnected-(U7-Pad21)
- U7 pad 22: Net-(U7-Pad22) -> unconnected-(U7-Pad22)
- U7 pad 3: Net-(U7-Pad3) -> unconnected-(U7-Pad3)
- U7 pad 4: Net-(U7-Pad4) -> unconnected-(U7-Pad4)
- U7 pad 5: Net-(U7-Pad5) -> unconnected-(U7-Pad5)
- U7 pad 6: Net-(U7-Pad6) -> unconnected-(U7-Pad6)
- U7 pad 7: Net-(U7-Pad7) -> unconnected-(U7-Pad7)
- U7 pad 8: Net-(U7-Pad8) -> unconnected-(U7-Pad8)
- U7 pad 9: Net-(U7-Pad9) -> unconnected-(U7-Pad9)
Other:
- net class Default removed
- board text added: "Left back"
- board text added: "Left front"
- board text added: "Right back"
- board text added: "Right front"

Commit message: new
Parts:
- added C103: 2200uF, Capacitor_THT:CP_Radial_D12.5mm_P5.00mm, F.Cu at (108.0, 194.7)
- added C104: 2200uF, Capacitor_THT:CP_Radial_D12.5mm_P5.00mm, F.Cu at (110.7, 183.8)
- added D10: TVS 3,6V, Diode_SMD:D_1206_3216Metric, F.Cu at (147.2, 194.5)
- added D11: TVS 6V, Diode_SMD:D_1206_3216Metric, F.Cu at (144.8, 186.2)
- added D12: TVS 15V, Diode_SMD:D_1206_3216Metric, F.Cu at (135.8, 166.8)
- added F2: Fuse, Fuse:Fuseholder_Cylinder-5x20mm_Schurter_0031_8201_Horizontal_Open, F.Cu at (69.6, 141.7)
- added F3: Fuse, Fuse:Fuseholder_Cylinder-5x20mm_Schurter_0031_8201_Horizontal_Open, F.Cu at (89.0, 169.4)
- C1, C2: value 4700uF -> 2200uF
- C11, C35, C36, C37, C38, C7, C8, C9: footprint Capacitor_THT:CP_Radial_D4.0mm_P2.00mm -> Capacitor_SMD:C_1206_3216Metric
- C13, C14, C25, C26, C47, C48, C49, C50: footprint Capacitor_THT:CP_Radial_D8.0mm_P2.50mm -> Capacitor_THT:CP_Radial_D12.5mm_P5.00mm
- C15, C17, C39, C40: footprint Capacitor_SMD:CP_Elec_4x3 -> Capacitor_THT:C_Radial_D8.0mm_H11.5mm_P3.50mm
- C16, C18, C41, C42: footprint Capacitor_THT:CP_Radial_D4.0mm_P2.00mm -> Capacitor_THT:C_Radial_D8.0mm_H11.5mm_P3.50mm
- C19, C20, C27, C28, C51, C52, C53, C54: footprint Capacitor_THT:CP_Radial_D8.0mm_P2.50mm -> Capacitor_THT:CP_Radial_D10.0mm_P5.00mm
- C80, C81, C82: footprint Capacitor_SMD:C_1206_3216Metric -> Capacitor_SMD:C_0805_2012Metric
- C92, C98: value C -> 100nF; footprint Capacitor_SMD:C_1206_3216Metric -> Capacitor_SMD:C_0805_2012Metric
- D1: footprint Diode_THT:D_DO-201AE_P12.70mm_Horizontal -> Diode_THT:D_DO-35_SOD27_P7.62mm_Horizontal
- D9: footprint LED_SMD:LED_1206_3216Metric -> LED_SMD:LED_0805_2012Metric
- K1: footprint Relay_THT:Relay_DPDT_FRT5 -> Relay_THT:Relay_DPDT_Fujitsu_FTR-F1C
- L1, L2: footprint Inductor_SMD:L_1206_3216Metric -> Inductor_SMD:L_0805_2012Metric
- R10, R11, R20, R21, R22, R23, R24, R25, R6, R7, R8, R9: footprint Resistor_THT:R_Axial_DIN0309_L9.0mm_D3.2mm_P15.24mm_Horizontal -> Resistor_THT:R_Axial_DIN0204_L3.6mm_D1.6mm_P7.62mm_Horizontal
- R12, R14, R26, R27: footprint Resistor_THT:R_Axial_DIN0207_L6.3mm_D2.5mm_P7.62mm_Horizontal -> Resistor_THT:R_Axial_DIN0204_L3.6mm_D1.6mm_P7.62mm_Horizontal
- moved H1 360.0 mm to (352.8, 202.5)
- moved D1 291.1 mm to (334.9, 137.8), turned to -90 degrees
- moved K1 275.2 mm to (328.5, 157.2)
- moved Q1 267.3 mm to (339.9, 139.6), turned to 180 degrees
- moved R1 267.3 mm to (339.9, 143.6), turned to 180 degrees
- moved HS2 214.4 mm to (300.0, 85.0)
- moved D9 201.7 mm to (283.2, 202.0)
- moved H6 200.9 mm to (67.5, 97.5)
- moved L1 178.2 mm to (257.2, 189.2), turned to -90 degrees
- moved C92 167.3 mm to (254.0, 196.0), turned to 180 degrees
- moved L2 160.3 mm to (254.0, 193.8)
- moved C98 157.6 mm to (257.0, 193.0), turned to 90 degrees
- moved C12 122.3 mm to (302.0, 138.8), turned to 90 degrees
- moved C76 116.2 mm to (270.5, 197.5), turned to 180 degrees
- moved C46 116.1 mm to (234.0, 139.2), turned to 90 degrees
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Connections:
- C1 pad 2: GNDPWR -> PWR_GND
- C10 pad 2: V-_3 -> -36V
- C12 pad 1: V+_3 -> +36V
- C13 pad 2: V-_3 -> -36V
- C14 pad 1: V+_3 -> +36V
- C19 pad 2: V-_3 -> -36V
- C2 pad 1: GNDPWR -> PWR_GND
- C20 pad 1: V+_3 -> +36V
- C21 pad 2: V-_4 -> -36V
- C22 pad 1: V+_4 -> +36V
- C23 pad 2: V-_3 -> -36V
- C24 pad 1: V+_3 -> +36V
- C25 pad 2: V-_4 -> -36V
- C26 pad 1: V+_4 -> +36V
- C27 pad 2: V-_4 -> -36V
- C28 pad 1: V+_4 -> +36V
- C29 pad 2: V-_4 -> -36V
- C30 pad 1: V+_4 -> +36V
- C43 pad 2: V-_2 -> -36V
- C44 pad 2: V-_1 -> -36V
- C45 pad 1: V+_2 -> +36V
- C46 pad 1: V+_1 -> +36V
- C47 pad 2: V-_2 -> -36V
- C48 pad 2: V-_1 -> -36V
- C49 pad 1: V+_2 -> +36V
- C50 pad 1: V+_1 -> +36V
- C51 pad 2: V-_2 -> -36V
- C52 pad 2: V-_1 -> -36V
- C53 pad 1: V+_2 -> +36V
- C54 pad 1: V+_1 -> +36V
- C55 pad 2: V-_2 -> -36V
- C56 pad 2: V-_1 -> -36V
- C57 pad 1: V+_2 -> +36V
- C58 pad 1: V+_1 -> +36V
- C88 pad 1: GNDD -> Net-(C85-Pad1)
- C94 pad +: (no net) -> +3V3
- D2 pad 3: /12Vac -> Net-(D2-Pad3)
- D2 pad 4: /12Vac -> Net-(D2-Pad4)
- D3 pad 1: GNDPWR -> PWR_GND
- D4 pad 2: GNDPWR -> PWR_GND
- R12 pad 1: V-_4 -> -36V
- R14 pad 1: V-_3 -> -36V
- R26 pad 1: V-_1 -> -36V
- R27 pad 1: V-_2 -> -36V
- R33 pad 2: GNDD -> Net-(C85-Pad1)
- R36 pad 2: GNDD -> Net-(C85-Pad1)
- U1 pad 1: V+_4 -> +36V
- U1 pad 4: V-_4 -> -36V
- U1 pad 5: V+_4 -> +36V
- U10 pad 3: GNDD -> Net-(C85-Pad1)
- U10 pad 4: (no net) -> +3V3
- U2 pad 1: V+_3 -> +36V
- U2 pad 4: V-_3 -> -36V
- U2 pad 5: V+_3 -> +36V
- U3 pad 1: V+_1 -> +36V
- U3 pad 4: V-_1 -> -36V
- U3 pad 5: V+_1 -> +36V
- U4 pad 1: V+_2 -> +36V
- U4 pad 4: V-_2 -> -36V
- U4 pad 5: V+_2 -> +36V
Routing:
- net -36V: track 0.00 -> 465.9 mm
- net PWR_GND: track 0.00 -> 414.4 mm, vias 0 -> 3
- net +36V: track 0.00 -> 414.1 mm
- net GNDD: track 0.00 -> 240.1 mm, vias 0 -> 4
- net +3V3: track 0.00 -> 211.6 mm, vias 0 -> 5
- net +15V: track 0.00 -> 65.5 mm
- net +5V: track 0.00 -> 57.2 mm
- net GNDA: track 0.00 -> 44.5 mm, vias 0 -> 1
- net Net-(C1-Pad1): track 0.00 -> 37.8 mm
- net SIG_GND: track 0.00 -> 30.0 mm
- net Net-(C2-Pad2): track 0.00 -> 29.4 mm
- net +12V: track 0.00 -> 21.0 mm
- net Net-(C83-Pad1): track 0.00 -> 20.7 mm
- net Net-(D5-Pad1): track 0.00 -> 20.4 mm
- net Net-(D8-Pad1): track 0.00 -> 19.8 mm
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- added copper zone on F.Cu, net (none)
- added copper zone on F.Cu, net +36V
- added copper zone on F.Cu, net -36V
- added copper zone on F.Cu, net GNDD
- added copper zone on F.Cu, net PWR_GND
Other:
- board size 250 x 100 mm -> 300 x 120 mm
- board text added: "+12 V"
- board text added: "+3,3 V"
- board text added: "+5 V"
- board text added: "zrobić dziurę w kształcie napisu"

Commit message: new
Parts:
- added C105: 100nF, Capacitor_SMD:C_1206_3216Metric, F.Cu at (333.2, 140.8)
- added C106: C, Capacitor_SMD:C_0805_2012Metric, F.Cu at (200.6, 157.3)
- added C107: C, Capacitor_SMD:C_0805_2012Metric, F.Cu at (203.5, 155.8)
- added C108: C, Capacitor_SMD:C_0805_2012Metric, F.Cu at (218.6, 172.2)
- added C109: C, Capacitor_SMD:C_0805_2012Metric, F.Cu at (221.7, 164.2)
- added C110: C, Capacitor_SMD:C_0805_2012Metric, F.Cu at (223.3, 159.0)
- added C111: C, Capacitor_SMD:C_0805_2012Metric, F.Cu at (211.8, 162.8)
- added C112: C, Capacitor_SMD:C_0805_2012Metric, F.Cu at (201.8, 172.4)
- added C113: C, Capacitor_SMD:C_0805_2012Metric, F.Cu at (232.9, 162.7)
- added C114: C, Capacitor_SMD:C_0805_2012Metric, F.Cu at (222.8, 173.0)
- added C115: C, Capacitor_SMD:C_0805_2012Metric, F.Cu at (211.8, 159.4)
- added C116: C, Capacitor_SMD:C_0805_2012Metric, F.Cu at (232.9, 159.3)
- added C117: C, Capacitor_SMD:C_0805_2012Metric, F.Cu at (209.9, 159.4)
- added C118: C, Capacitor_SMD:C_0805_2012Metric, F.Cu at (230.9, 159.3)
- added C119: C, Capacitor_SMD:C_0805_2012Metric, F.Cu at (208.3, 172.3)
- added C120: C, Capacitor_SMD:C_0805_2012Metric, F.Cu at (229.1, 172.2)
- added C121: C, Capacitor_SMD:C_0805_2012Metric, F.Cu at (207.1, 157.8)
- added C122: C, Capacitor_SMD:C_0805_2012Metric, F.Cu at (228.1, 157.8)
- added C123: C, Capacitor_SMD:C_0805_2012Metric, F.Cu at (205.3, 170.8)
- added C124: C, Capacitor_SMD:C_0805_2012Metric, F.Cu at (226.2, 170.9)
- added C125: C, Capacitor_SMD:C_0805_2012Metric, F.Cu at (209.9, 169.3)
- added C126: C, Capacitor_SMD:C_0805_2012Metric, F.Cu at (230.9, 169.1)
- added C127: C, Capacitor_SMD:C_0805_2012Metric, F.Cu at (200.2, 178.1)
- added C128: C, Capacitor_SMD:C_0805_2012Metric, F.Cu at (211.6, 177.4)
- added C129: C, Capacitor_SMD:C_0805_2012Metric, F.Cu at (213.8, 177.4)
- added C130: C, Capacitor_SMD:C_0805_2012Metric, F.Cu at (217.7, 179.2)
- added C131: C, Capacitor_SMD:C_0805_2012Metric, F.Cu at (202.2, 181.6)
- added C132: C, Capacitor_SMD:C_0805_2012Metric, F.Cu at (217.8, 181.1)
- added C133: C, Capacitor_SMD:C_0805_2012Metric, F.Cu at (220.1, 186.4)
- added C134: C, Capacitor_SMD:C_0805_2012Metric, F.Cu at (233.4, 182.3)
- added C135: C, Capacitor_SMD:C_0805_2012Metric, F.Cu at (218.8, 183.6)
- added C136: C, Capacitor_SMD:C_0805_2012Metric, F.Cu at (205.5, 181.7)
- added C137: C, Capacitor_SMD:C_0805_2012Metric, F.Cu at (210.2, 185.8)
- added C138: C, Capacitor_SMD:C_0805_2012Metric, F.Cu at (239.8, 160.6)
- added C139: 100nF, Capacitor_SMD:C_0805_2012Metric, F.Cu at (285.3, 169.3)
- added F1: Fuse, Fuse:Fuse_1206_3216Metric, F.Cu at (122.1, 182.0)
- added J1: AudioJack3, Connector_Audio:Jack_3.5mm_CUI_SJ1-3533NG_Horizontal, F.Cu at (177.0, 206.0)
- added J2: AudioJack3, Connector_Audio:Jack_3.5mm_CUI_SJ1-3533NG_Horizontal, F.Cu at (127.0, 206.0)
- added J3: USB_A, amplituner_lib:usb_A, F.Cu at (332.1, 200.5)
- added J4: Conn_01x03, Connector_PinHeader_2.54mm:PinHeader_1x03_P2.54mm_Vertical, F.Cu at (265.2, 157.7)
- added J5: Conn_02x02_Counter_Clockwise, Connector_PinHeader_2.54mm:PinHeader_2x02_P2.54mm_Vertical, F.Cu at (194.0, 204.0)
- added J6: Conn_02x03_Counter_Clockwise, Connector_PinHeader_2.54mm:PinHeader_2x03_P2.54mm_Vertical, F.Cu at (186.7, 201.5)
- added J7: Conn_02x03_Counter_Clockwise, Connector_PinHeader_2.54mm:PinHeader_2x03_P2.54mm_Vertical, F.Cu at (200.9, 201.4)
- added R41: R, Resistor_SMD:R_0805_2012Metric, F.Cu at (197.8, 170.2)
- added R42: R, Resistor_SMD:R_0805_2012Metric, F.Cu at (219.4, 167.7)
- added R43: R, Resistor_SMD:R_0805_2012Metric, F.Cu at (218.5, 170.3)
- added R44: R, Resistor_SMD:R_0805_2012Metric, F.Cu at (209.9, 165.9)
- added R45: R, Resistor_SMD:R_0805_2012Metric, F.Cu at (209.9, 162.8)
- added R46: R, Resistor_SMD:R_0805_2012Metric, F.Cu at (230.9, 165.7)
- added R47: R, Resistor_SMD:R_0805_2012Metric, F.Cu at (230.9, 162.7)
- added R48: R, Resistor_SMD:R_0805_2012Metric, F.Cu at (200.9, 170.1)
- added R49: R, Resistor_SMD:R_0805_2012Metric, F.Cu at (221.9, 170.3)
- added R50: R, Resistor_SMD:R_0805_2012Metric, F.Cu at (201.8, 167.6)
- added R51: R, Resistor_SMD:R_0805_2012Metric, F.Cu at (213.8, 162.8)
- added R52: R, Resistor_SMD:R_0805_2012Metric, F.Cu at (222.8, 167.6)
- added R53: R, Resistor_SMD:R_0805_2012Metric, F.Cu at (234.9, 162.7)
- added R54: R, Resistor_SMD:R_0805_2012Metric, F.Cu at (213.8, 158.2)
- added R55: R, Resistor_SMD:R_0805_2012Metric, F.Cu at (234.9, 158.1)
- added R56: R, Resistor_SMD:R_0805_2012Metric, F.Cu at (210.5, 156.3)
- added R57: R, Resistor_SMD:R_0805_2012Metric, F.Cu at (231.5, 156.5)
- added R58: R, Resistor_SMD:R_0805_2012Metric, F.Cu at (205.3, 173.2)
- added R59: R, Resistor_SMD:R_0805_2012Metric, F.Cu at (226.2, 173.1)
- added R60: R, Resistor_SMD:R_0805_2012Metric, F.Cu at (207.1, 159.7)
- added R61: R, Resistor_SMD:R_0805_2012Metric, F.Cu at (228.1, 159.5)
- added R62: R, Resistor_SMD:R_0805_2012Metric, F.Cu at (205.3, 169.1)
- added R63: R, Resistor_SMD:R_0805_2012Metric, F.Cu at (226.2, 168.9)
- added R64: R, Resistor_SMD:R_0805_2012Metric, F.Cu at (204.9, 178.8)
- added R65: R, Resistor_SMD:R_0805_2012Metric, F.Cu at (202.2, 178.1)
- added R66: R, Resistor_SMD:R_0805_2012Metric, F.Cu at (220.8, 177.2)
- added R67: R, Resistor_SMD:R_0805_2012Metric, F.Cu at (217.7, 177.2)
- added R68: R, Resistor_SMD:R_0805_2012Metric, F.Cu at (200.2, 181.6)
- added R69: R, Resistor_SMD:R_0805_2012Metric, F.Cu at (208.8, 178.2)
- added R70: R, Resistor_SMD:R_0805_2012Metric, F.Cu at (221.1, 179.2)
- added R71: R, Resistor_SMD:R_0805_2012Metric, F.Cu at (223.9, 180.0)
- added R72: R, Resistor_SMD:R_0805_2012Metric, F.Cu at (220.9, 183.5)
- added R73: R, Resistor_SMD:R_0805_2012Metric, F.Cu at (233.4, 180.3)
- added R74: R, Resistor_SMD:R_0805_2012Metric, F.Cu at (216.9, 183.6)
- added R75: R, Resistor_SMD:R_0805_2012Metric, F.Cu at (207.4, 181.7)
- added R76: R, Resistor_SMD:R_1206_3216Metric, F.Cu at (274.0, 177.4)
- added R77: R, Resistor_SMD:R_1206_3216Metric, F.Cu at (266.8, 183.2)
- added SW1: NRST_BUTT, Button_Switch_SMD:SW_SPST_FSMSM, F.Cu at (247.1, 159.3)
- added U12: bluetooth_module, amplituner_lib:bluetooth_module, F.Cu at (346.8, 156.4)
- added U13: LM833D, amplituner_lib:LMV358, F.Cu at (205.6, 164.3)
- added U14: LM833D, amplituner_lib:LMV358, F.Cu at (226.5, 164.1)
- added U15: LM833D, amplituner_lib:LMV358, F.Cu at (212.2, 181.9)
- added U16: CS43L21, Package_DFN_QFN:QFN-32-1EP_5x5mm_P0.5mm_EP3.45x3.45mm, F.Cu at (284.4, 183.2)
- added U17: CAT24C256, amplituner_lib:CAT24C256, F.Cu at (286.7, 165.1)
- added U18: USBLC6-4SC6, Package_TO_SOT_SMD:SOT-23-6, F.Cu at (332.0, 193.2)
- C61, C67, C68, C69: value 100nF -> 4,7uF; footprint Capacitor_SMD:C_1206_3216Metric -> Capacitor_SMD:CP_Elec_6.3x5.2
- R30: footprint Resistor_SMD:R_1206_3216Metric -> Resistor_SMD:R_0805_2012Metric
- Y1: footprint Crystal:Crystal_HC52-6mm_Vertical -> Crystal:Crystal_SMD_HC49-SD
- moved Q1 313.6 mm to (29.0, 98.6), turned to -90 degrees
- moved R1 310.2 mm to (33.0, 98.6), turned to -90 degrees
- moved D1 309.6 mm to (27.2, 103.6), turned to 0 degrees
- moved K1 286.4 mm to (48.4, 97.3), turned to -90 degrees
- moved L3 90.7 mm to (224.6, 196.6), turned to 180 degrees
- moved C100 81.8 mm to (237.4, 190.2)
- moved C101 80.1 mm to (229.8, 196.6)
- moved C99 74.4 mm to (237.4, 187.2)
- moved C102 73.9 mm to (229.7, 193.5)
- moved R30 73.6 mm to (198.7, 167.8), turned to 90 degrees
- moved L4 73.5 mm to (224.5, 193.5), turned to 180 degrees
- moved C82 72.5 mm to (197.8, 171.8), turned to 180 degrees
- moved U11 66.9 mm to (239.3, 196.6), turned to 180 degrees
- moved C61 66.5 mm to (136.1, 197.9), turned to -90 degrees
- moved R31 64.6 mm to (193.9, 198.9), turned to 90 degrees
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Connections:
- C82 pad 1: POWER_BUTTON -> Net-(R30-Pad1)
- C82 pad 2: GNDD -> GNDA
- C94 pad +: +3V3 -> (no net)
- D10 pad 1: +3V3 -> (no net)
- L3 pad 2: Radio_in_L -> Radio_L
- L4 pad 2: Radio_in_R -> Radio_R
- Q2 pad 3: Net-(D9-Pad1) -> Net-(J5-Pad3)
- R30 pad 1: POWER_BUTTON -> Net-(R30-Pad1)
- R30 pad 2: Net-(R30-Pad2) -> +3V3
- U10 pad 4: +3V3 -> (no net)
- U5 pad 16: unconnected-(U5-Pad16) -> AUDIO_IN_SubR
- U5 pad 17: unconnected-(U5-Pad17) -> AUDIO_IN_SubL
- U6 pad 10: SPI3_CD -> SPI3_CS
- U6 pad 44: unconnected-(U6-Pad44) -> MCU_USB_DM
- U6 pad 45: unconnected-(U6-Pad45) -> MCU_USB_DP
Routing:
- net AUDIO_IN_LB: track 0.00 -> 199.5 mm
- net I2C_SDA: track 0.00 -> 177.5 mm, vias 0 -> 4
- net I2C_SCL: track 0.00 -> 162.7 mm, vias 0 -> 2
- net +5V: track 57.2 -> 204.8 mm, vias 0 -> 1
- net AUDIO_IN_LF: track 0.00 -> 136.2 mm, vias 0 -> 3
- net AUDIO_IN_RB: track 0.00 -> 135.9 mm, vias 0 -> 5
- net AUDIO_IN_RF: track 0.00 -> 111.4 mm, vias 0 -> 5
- net GNDD: track 240.1 -> 132.6 mm, vias 4 -> 2
- net Net-(C61-Pad1): track 0.00 -> 55.2 mm, vias 0 -> 2
- net GNDA: track 44.5 -> 95.7 mm, vias 1 -> 2
- net Net-(C67-Pad1): track 0.00 -> 47.9 mm, vias 0 -> 2
- net Net-(C60-Pad1): track 0.00 -> 37.5 mm
- net Net-(C68-Pad1): track 0.00 -> 34.2 mm
- net Jack_1_IN_G: track 0.00 -> 32.8 mm
- net Net-(C69-Pad1): track 0.00 -> 31.4 mm
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- added copper zone on F.Cu, net +12V
- added copper zone on F.Cu, net +15V
- added copper zone on F.Cu, net GNDA
- added copper zone on F.Cu, net Net-(C84-Pad1)
Other:
- outline, holes or cut-outs redrawn
- board text added: "+36V"
- board text added: "-36V"
- board text added: "12Vac"
- board text added: "24Vac"
- board text added: "Left back input"
- board text added: "Left front input"
- board text added: "NRST"
- board text added: "Right back input"
- board text added: "Right front input"
- board text added: "SWCLK"
- board text added: "SWDIO"
- board text added: "zrobić dziurę w kształcie napisu dodać znak wodny dodać swój rysunek i podpis Nazwę w jednym miejscu W drugim (c) 2022 Maciej Kotowicz"
- board text removed: "Left front"
- board text removed: "zrobić dziurę w kształcie napisu"

Commit message: new
Parts:
- removed C63, C70: 100nF, Capacitor_SMD:C_1206_3216Metric
- removed D9: LED, LED_SMD:LED_0805_2012Metric
- moved Q2 83.1 mm to (196.9, 200.1), turned to 180 degrees
- moved C134 32.5 mm to (201.0, 184.9)
- moved R73 29.6 mm to (204.2, 184.9), turned to 0 degrees
- moved J6 15.3 mm to (202.0, 201.4)
- moved J7 14.5 mm to (186.4, 201.4)
- moved C71 13.5 mm to (181.8, 188.5)
- moved C64 9.22 mm to (186.7, 188.5), turned to 180 degrees
- moved C133 8.64 mm to (225.9, 180.0), turned to -90 degrees
- moved C105 7.80 mm to (333.4, 148.6)
- moved U12 7.40 mm to (346.9, 163.8)
- moved J5 3.61 mm to (196.7, 206.4), turned to 180 degrees
- moved R72 1.27 mm to (221.8, 182.6), turned to 180 degrees
- moved C77 1.00 mm to (255.3, 180.3)
- moved C80 0.85 mm to (246.4, 168.5)
- moved C81 0.85 mm to (246.4, 172.2)
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Connections:
- net Net-(C135-Pad2) renamed ADC2_SUB1
- net Net-(C136-Pad2) renamed ADC2_SUB2
- C82 pad 1: Net-(R30-Pad1) -> GNDA
- C82 pad 2: GNDA -> Net-(R30-Pad1)
- C94 pad +: (no net) -> +3V3
- D10 pad 1: (no net) -> +3V3
- U10 pad 4: (no net) -> +3V3
- U5 pad 10: Net-(C63-Pad1) -> Radio_L
- U5 pad 11: Net-(C70-Pad1) -> Radio_R
- U6 pad 16: ADC2_IN7 -> ADC2_IN12
- U6 pad 17: ADC2_IN8 -> ADC2_IN13
- U6 pad 23: ADC2_IN12 -> ADC2_IN7
- U6 pad 24: ADC2_IN13 -> ADC2_IN8
Routing:
- net +5V: track 204.8 -> 294.0 mm, vias 1 -> 2
- net ADC2_IN8: track 4.04 -> 69.9 mm, vias 0 -> 4
- net ADC2_IN7: track 4.47 -> 67.5 mm, vias 0 -> 4
- net Radio_L: track 0.00 -> 59.9 mm, vias 0 -> 2
- net Radio_R: track 0.00 -> 57.8 mm, vias 0 -> 2
- net ADC2_SUB2: track 4.24 -> 51.9 mm, vias 0 -> 2
- net AUDIO_IN_SubL: track 5.66 -> 50.9 mm
- net ADC2_IN13: track 4.34 -> 43.4 mm, vias 0 -> 2
- net ADC2_SUB1: track 4.40 -> 42.9 mm, vias 0 -> 2
- net ADC2_IN12: track 4.25 -> 38.5 mm, vias 0 -> 2
- net AUDIO_IN_SubR: track 18.4 -> 46.6 mm
- net +3V3: track 226.6 -> 244.2 mm, vias 8 -> 11
- net Net-(C64-Pad1): track 0.00 -> 17.2 mm
- net Net-(C71-Pad1): track 0.00 -> 15.7 mm
- net POWER_BUTTON: track 0.00 -> 15.4 mm
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