File: Hardware/kicad/block diagram/block-sch/block-sch.kicad_pcb (KiCad board)
At the start: 2 copper layers, 300 x 120 mm, 381 parts, among them J1 AudioJack3, J10 Conn_02x02_Counter_Clockwise, J11 Conn_02x02_Counter_Clockwise, J12 Conn_02x02_Counter_Clockwise, J13 Conn_02x03_Counter_Clockwise, J14 Conn_02x03_Counter_Clockwise, J15 Conn_01x02, J16 Conn_01x03, J17 AudioJack3, J18 Conn_01x03, J19 Conn_01x03, J2 AudioJack3, J20 AudioJack3, J3 USB_A, J4 Conn_01x03, J5 Conn_02x02_Counter_Clockwise, J6 Conn_02x02_Counter_Clockwise, J7 Conn_02x02_Counter_Clockwise, J8 Conn_02x02_Counter_Clockwise, J9 Conn_02x02_Counter_Clockwise, K1 AZ850-x, K2 G6K-2, K3 G6K-2, K4 G6K-2, Q1 BC817, Q2 BC817, Q3 BC817, SW1 NRST_BUTT, U1 LM3886, U10 AZ1117-3.3, U11 RDA5807M, U12 bluetooth_module, U13 LM833D, U14 LM833D, U15 LM833D, U16 CS43L21, U17 CAT24C256, U18 USBLC6-4SC6, U19 LM78M05_TO252, U2 LM3886, U20 LM833D, U21 LM833D, U3 LM3886, U4 LM3886, U5 TDA7719, U6 STM32L4Q5, U7 ESP8266-12E_ESP-12E, U8 LM7812_TO220, U9 LM78M05_TO252, Y1 Crystal

Commit message: new
Parts:
- moved R82 33.7 mm to (253.6, 201.1), turned to 0 degrees
- moved R78 32.0 mm to (250.2, 202.9), turned to 180 degrees
- moved J6 31.9 mm to (251.3, 206.9)
- moved R86 31.7 mm to (253.6, 203.0), turned to 0 degrees
- moved R89 9.86 mm to (245.8, 202.9), turned to 0 degrees
- moved J9 9.35 mm to (243.5, 206.8)
- moved R81 9.26 mm to (242.5, 202.9), turned to 180 degrees
- moved R95 8.17 mm to (222.2, 200.9), turned to 0 degrees
- moved R85 8.00 mm to (245.9, 200.9), turned to 0 degrees
- moved R124 7.12 mm to (231.9, 173.4), turned to 90 degrees
- moved R92 6.50 mm to (218.8, 202.9), turned to 180 degrees
- moved J12 6.41 mm to (219.9, 206.8)
- moved R94 6.39 mm to (214.4, 200.9), turned to 0 degrees
- moved R98 6.10 mm to (222.2, 202.9), turned to 0 degrees
- moved U11 5.31 mm to (242.7, 189.3)
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Connections:
- J10 pad 3: TIM3_CH2 -> ENC_MIDDLE_2
- J10 pad 4: TIM3_CH1 -> ENC_MIDDLE_1
- J11 pad 3: TIM5_CH2 -> ENC_TREBLE_2
- J11 pad 4: TIM5_CH1 -> ENC_TREBLE_1
- J12 pad 3: TIM4_CH2 -> ENC_BASS_2
- J12 pad 4: TIM4_CH1 -> ENC_BASS_1
- J6 pad 3: TIM8_CH2 -> ENC_VOL_BACK_1
- J6 pad 4: TIM8_CH1 -> ENC_VOL_BACK_2
- J7 pad 3: TIM1_CH2 -> ENC_LOUD_2
- J7 pad 4: TIM1_CH1 -> ENC_LOUD_1
- J8 pad 3: TIM2_CH2 -> ENC_VOL_FRONT_2
- J8 pad 4: TIM2_CH1 -> ENC_VOL_FRONT_1
- J9 pad 3: Net-(J9-Pad3) -> ENC_RADIO_2
- J9 pad 4: Net-(J9-Pad4) -> ENC_RADIO_1
- R82 pad 2: TIM8_CH1 -> ENC_VOL_BACK_2
- R83 pad 2: TIM1_CH1 -> ENC_LOUD_1
- R84 pad 2: TIM2_CH1 -> ENC_VOL_FRONT_1
- R85 pad 2: Net-(J9-Pad4) -> ENC_RADIO_1
- R86 pad 2: TIM8_CH2 -> ENC_VOL_BACK_1
- R87 pad 2: TIM1_CH2 -> ENC_LOUD_2
- R88 pad 2: TIM2_CH2 -> ENC_VOL_FRONT_2
- R89 pad 2: Net-(J9-Pad3) -> ENC_RADIO_2
- R93 pad 2: TIM3_CH1 -> ENC_MIDDLE_1
- R94 pad 2: TIM5_CH1 -> ENC_TREBLE_1
- R95 pad 2: TIM4_CH1 -> ENC_BASS_1
- R96 pad 2: TIM3_CH2 -> ENC_MIDDLE_2
- R97 pad 2: TIM5_CH2 -> ENC_TREBLE_2
- R98 pad 2: TIM4_CH2 -> ENC_BASS_2
- U6 pad 50: ENC_VOL_FRON_1 -> ENC_VOL_FRONT_1
- U6 pad 54: END_RADIO_1 -> ENC_RADIO_1
- U6 pad 57: END_MIDDLE_2 -> ENC_MIDDLE_2
- U6 pad 59: ENC_BAS_2 -> ENC_BASS_2
Routing:
- net +5V: track 197.4 -> 80.1 mm
- net SPI3_SCK: track 0.00 -> 95.8 mm, vias 0 -> 1
- net SPI3_MOSI: track 0.00 -> 93.0 mm, vias 0 -> 1
- net SPI3_DC: track 0.00 -> 87.2 mm, vias 0 -> 1
- net SPI3_CS: track 0.00 -> 83.4 mm, vias 0 -> 1
- net ENC_BUT_TREBLE: track 0.00 -> 79.1 mm, vias 0 -> 1
- net ENC_BUT_BASS: track 0.00 -> 65.9 mm, vias 0 -> 1
- net ENC_BASS_2: track 0.00 -> 61.0 mm, vias 0 -> 1
- net ENC_MIDDLE_2: track 0.00 -> 55.1 mm, vias 0 -> 1
- net ENC_BASS_1: track 0.00 -> 54.2 mm, vias 0 -> 2
- net ENC_MIDDLE_1: track 0.00 -> 48.3 mm, vias 0 -> 2
- net ENC_VOL_FRONT_2: track 0.00 -> 44.9 mm, vias 0 -> 1
- net ENC_VOL_FRONT_1: track 0.00 -> 42.6 mm, vias 0 -> 2
- net ENC_BUT_VOL_FRONT: track 11.1 -> 48.0 mm
- net ENC_VOL_BACK_1: track 9.46 -> 44.9 mm
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
Commit message: new
Parts:
- removed D1, D17, D18, D19: D, Diode_THT:D_DO-35_SOD27_P7.62mm_Horizontal
- removed D9: TVS 3,6V, Diode_SMD:D_1206_3216Metric
- removed K1: AZ850-x, Relay_THT:Relay_DPDT_Fujitsu_FTR-F1C
- removed Q1: BC817, Package_TO_SOT_SMD:SOT-23
- removed R1: R, Resistor_SMD:R_1206_3216Metric
- added R126: R, Resistor_SMD:R_0805_2012Metric, F.Cu at (190.1, 202.8)
- added R127: R, Resistor_SMD:R_0805_2012Metric, F.Cu at (193.6, 202.8)
- added R128: R, Resistor_SMD:R_0805_2012Metric, F.Cu at (190.2, 200.8)
- added R129: R, Resistor_SMD:R_0805_2012Metric, F.Cu at (193.6, 200.8)
- R106: footprint Resistor_SMD:R_1206_3216Metric -> Resistor_SMD:R_0805_2012Metric
- moved C140 61.4 mm to (238.9, 174.2), turned to 90 degrees
- moved R105 60.4 mm to (235.6, 175.6)
- moved D16 59.1 mm to (235.2, 173.4)
- moved C162 31.1 mm to (314.5, 187.5), turned to 90 degrees
- moved R102 29.8 mm to (351.4, 132.7), turned to 180 degrees
- moved C163 29.5 mm to (307.1, 187.4)
- moved C60 21.9 mm to (172.5, 188.8), turned to -90 degrees
- moved R99 21.7 mm to (344.4, 153.5), turned to 180 degrees
- moved C65 17.7 mm to (169.7, 188.6), turned to -90 degrees
- moved R103 16.2 mm to (337.5, 153.5), turned to 180 degrees
- moved R107 15.0 mm to (284.8, 172.3), turned to 180 degrees
- moved C159 14.5 mm to (296.5, 184.6), turned to -90 degrees
- moved R108 13.6 mm to (285.2, 191.5), turned to 0 degrees
- moved C154 13.2 mm to (289.5, 190.5)
- moved R101 11.9 mm to (340.9, 153.5), turned to 180 degrees
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Connections:
- C59 pad 1: Net-(C59-Pad1) -> Net-(U5-Pad6)
- C59 pad 2: Jack_1_IN_R -> DAC_R
- C60 pad 1: Net-(C60-Pad1) -> Net-(U5-Pad7)
- C60 pad 2: Jack_2_IN_R -> Bluetooth_IN_L
- C61 pad 1: Net-(C61-Pad1) -> Net-(U5-Pad1)
- C61 pad 2: DAC_R -> Jack_1_IN_L
- C65 pad 1: Net-(C65-Pad1) -> Net-(U5-Pad5)
- C65 pad 2: Jack_1_IN_L -> DAC_L
- C66 pad 2: Jack_2_IN_L -> Bluetooth_IN_R
- C67 pad 1: Net-(C67-Pad1) -> Net-(U5-Pad2)
- C67 pad 2: DAC_L -> Jack_1_IN_R
- C68 pad 1: Net-(C68-Pad1) -> Net-(U5-Pad3)
- C68 pad 2: Bluetooth_IN_L -> Jack_2_IN_L
- C69 pad 1: Net-(C69-Pad1) -> Net-(U5-Pad4)
- C69 pad 2: Bluetooth_IN_R -> Jack_2_IN_R
- J13 pad 4: SPI3_DC -> SPI3_CS
- J13 pad 6: SPI3_CS -> SPI3_DC
- J14 pad 4: GNDD -> unconnected-(J14-Pad4)
- U5 pad 1: Net-(C65-Pad1) -> Net-(U5-Pad1)
- U5 pad 2: Net-(C59-Pad1) -> Net-(U5-Pad2)
- U5 pad 3: Net-(C66-Pad1) -> Net-(U5-Pad3)
- U5 pad 4: Net-(C60-Pad1) -> Net-(U5-Pad4)
- U5 pad 5: Net-(C67-Pad1) -> Net-(U5-Pad5)
- U5 pad 6: Net-(C61-Pad1) -> Net-(U5-Pad6)
- U5 pad 7: Net-(C68-Pad1) -> Net-(U5-Pad7)
- U5 pad 9: Net-(C69-Pad1) -> Net-(C66-Pad1)
Routing:
- net UART_RX: track 3.04 -> 124.7 mm, vias 1 -> 5
- net UART_TX: track 1.90 -> 120.0 mm, vias 1 -> 5
- net USER_BUTTON_1: track 18.5 -> 96.7 mm, vias 0 -> 2
- net USER_BUTTON_2: track 19.2 -> 94.3 mm, vias 0 -> 1
- net POWER_BUTTON: track 31.7 -> 106.0 mm, vias 0 -> 2
- net USER_BUTTON_3: track 20.9 -> 92.9 mm, vias 0 -> 2
- net USER_BUTTON_4: track 21.8 -> 87.1 mm, vias 0 -> 1
- net TIM16_CH1: track 17.4 -> 81.4 mm, vias 0 -> 2
- net ENC_TREBLE_1: track 11.7 -> 66.2 mm, vias 1 -> 4
- net +5V: track 80.1 -> 29.1 mm, vias 1 -> 2
- net +3V3: track 250.4 -> 300.0 mm, vias 8 -> 19
- net ENC_TREBLE_2: track 18.2 -> 64.9 mm, vias 0 -> 4
- net Headphones_in_G: track 0.00 -> 46.6 mm
- net I2C_SCL: track 161.5 -> 206.2 mm, vias 4 -> 8
- net Net-(U5-Pad2): track 0.00 -> 44.3 mm
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- added copper zone on F.Cu, net +3V3
- added copper zone on F.Cu, net ADC2_IN12
- added copper zone on F.Cu, net GNDA
- added copper zone on F.Cu, net Net-(C108-Pad2)
- added copper zone on F.Cu, net Net-(C109-Pad2)
- added copper zone on F.Cu, net Net-(C111-Pad2)
- added copper zone on F.Cu, net Net-(C113-Pad2)
- added copper zone on F.Cu, net Net-(C127-Pad2)
- added copper zone on F.Cu, net Net-(C130-Pad2)
- added copper zone on F.Cu, net Net-(C134-Pad2)
- added copper zone on F.Cu, net Net-(C161-Pad2)
- added copper zone on F.Cu, net Net-(C82-Pad2)
- removed copper zone on F.Cu, net Jack_1_IN_G
