File: Hardware/kicad/block diagram/block-sch/enc_butt_scheet.kicad_sch (KiCad schematic)
At the start: 0 parts

Commit message: new
Parts:
- added J? (x7): Conn_02x02_Counter_Clockwise, Connector_PinHeader_1.27mm:PinHeader_2x02_P1.27mm_Vertical, symbol Connector_Generic:Conn_02x02_Counter_Clockwise
- added J? (x2): Conn_02x03_Counter_Clockwise, Connector_PinHeader_1.27mm:PinHeader_2x03_P1.27mm_Vertical, symbol Connector_Generic:Conn_02x03_Counter_Clockwise
- added R? (x21): R, Resistor_SMD:R_0805_2012Metric, symbol Device:R
Connections:
- new net: J?.4 (Pin_4), R?.2
- new net: J?.3 (Pin_3), R?.2
- new net +3V3: R?.1, R?.1, R?.1, R?.1, R?.1, R?.1, R?.1, R?.1, R?.1, R?.1, R?.1, R?.1, R?.1, R?.1, R?.1, R?.1, R?.1, R?.1, R?.1, R?.1, R?.1
- new net ENC_BUT_BASS: J?.1 (Pin_1), R?.2
- new net ENC_BUT_LOUD: J?.1 (Pin_1), R?.2
- new net ENC_BUT_MIDDLE: J?.1 (Pin_1), R?.2
- new net ENC_BUT_RADIO: J?.1 (Pin_1), R?.2
- new net ENC_BUT_TREBLE: J?.1 (Pin_1), R?.2
- new net ENC_BUT_VOL_BACK: J?.1 (Pin_1), R?.2
- new net ENC_BUT_VOL_FRONT: J?.1 (Pin_1), R?.2
- new net GNDD: J?.2 (Pin_2), J?.2 (Pin_2), J?.2 (Pin_2), J?.2 (Pin_2), J?.2 (Pin_2), J?.2 (Pin_2), J?.2 (Pin_2), J?.3 (Pin_3), J?.4 (Pin_4)
- new net SP3_RESET: J?.5 (Pin_5)
- new net SPI3_CS: J?.6 (Pin_6)
- new net SPI3_DC: J?.4 (Pin_4)
- new net SPI3_MOSI: J?.2 (Pin_2)
- new net SPI3_SCK: J?.1 (Pin_1)
- new net TIM1_CH1: J?.4 (Pin_4), R?.2
- new net TIM1_CH2: J?.3 (Pin_3), R?.2
- new net TIM2_CH1: J?.4 (Pin_4), R?.2
- new net TIM2_CH2: J?.3 (Pin_3), R?.2
- new net TIM3_CH1: J?.4 (Pin_4), R?.2
- new net TIM3_CH2: J?.3 (Pin_3), R?.2
- new net TIM4_CH1: J?.4 (Pin_4), R?.2
- new net TIM4_CH2: J?.3 (Pin_3), R?.2
- new net TIM5_CH1: J?.4 (Pin_4), R?.2
- new net TIM5_CH2: J?.3 (Pin_3), R?.2
- new net TIM8_CH1: J?.4 (Pin_4), R?.2
- new net TIM8_CH2: J?.3 (Pin_3), R?.2
- new net USER_BUTTON_1: J?.2 (Pin_2)
- new net USER_BUTTON_2: J?.6 (Pin_6)
- new net USER_BUTTON_3: J?.1 (Pin_1)
- new net USER_BUTTON_4: J?.5 (Pin_5)

Commit message: new
Parts:
- gave numbers to parts that had none: 30

Commit message: new
Connections:
- net ENC_RADIO_1: now reaches J9.4 (Pin_4), R85.2
- net ENC_RADIO_2: now reaches J9.3 (Pin_3), R89.2
- net TIM1_CH1 renamed ENC_LOUD_1
- net TIM1_CH2 renamed ENC_LOUD_2
- net TIM2_CH1 renamed ENC_VOL_FRONT_1
- net TIM2_CH2 renamed ENC_VOL_FRONT_2
- net TIM3_CH1 renamed ENC_MIDDLE_1
- net TIM3_CH2 renamed ENC_MIDDLE_2
- net TIM4_CH1 renamed ENC_BASS_1
- net TIM4_CH2 renamed ENC_BASS_2
- net TIM5_CH1 renamed ENC_TREBLE_1
- net TIM5_CH2 renamed ENC_TREBLE_2
- net TIM8_CH1 renamed ENC_VOL_BACK_2
- net TIM8_CH2 renamed ENC_VOL_BACK_1

Commit message: new
Parts:
- added R126, R127, R128, R129: R, Resistor_SMD:R_0805_2012Metric, symbol Device:R
Connections:
- net +3V3: now also R126.1, R127.1, R128.1, R129.1
- net GNDD: no longer J14.4 (Pin_4)
- net SPI3_CS: now also J13.4 (Pin_4); no longer J13.6 (Pin_6)
- net SPI3_DC: now also J13.6 (Pin_6); no longer J13.4 (Pin_4)
- net USER_BUTTON_1: now also R126.2
- net USER_BUTTON_2: now also R128.2
- net USER_BUTTON_3: now also R127.2
- net USER_BUTTON_4: now also R129.2
