File: Hardware/kicad/block diagram/block-sch/low_power_scheet.kicad_sch (KiCad schematic)
At the start: 32 parts, among them U10 AZ1117-3.3, U8 LM7812_TO220, U9 LM78M05_TO252

Commit message: new
Parts:
- D10, D11, D12: footprint (none) -> Diode_SMD:D_1206_3216Metric
Connections:
- net +3V3: now also D10.C
- net GNDD: no longer C85.1, C88.1, D10.C, R33.2, R36.2, U10.3 (VI)
- new net: C85.1, C88.1, R33.2, R36.2, U10.3 (VI)
Other:
- moved on the sheet: C85, C88, C91, C97, D10, D12, D15, R40

Commit message: new
Parts:
- added C140, C70: 100nF, Capacitor_SMD:C_1206_3216Metric, symbol Device:C
- added D16: LED, LED_SMD:LED_1206_3216Metric, symbol Device:LED
- added D9: TVS 3,6V, Diode_SMD:D_1206_3216Metric, symbol lib_amplituner:1SMB5914BT3G
- added R104, R105: R, Resistor_SMD:R_1206_3216Metric, symbol Device:R
- added U19: LM78M05_TO252, Package_TO_SOT_SMD:TO-252-2, symbol Regulator_Linear:LM78M05_TO252
Connections:
- net +3V3: now also R104.1
- net GNDD: now also C140.2, C70.2, D16.1 (K), D9.A, U19.2 (GND)
- new net: D16.2 (A), R105.1
- new net: C70.1, R104.2, U19.1 (VI)
- new net +1V8: C140.1, D9.C, R105.2, U19.3 (VO)

Commit message: new
Parts:
- C140, C70: footprint Capacitor_SMD:C_1206_3216Metric -> Capacitor_SMD:C_0805_2012Metric
- R104, R105: footprint Resistor_SMD:R_1206_3216Metric -> Resistor_SMD:R_0805_2012Metric
Changed lines of the file:
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@@
       (effects (font (size 1.27 1.27)) (justify left))
     )
-    (property "Footprint" "Capacitor_SMD:C_1206_3216Metric" (id 2) (at 143.3322 169.291 0)
+    (property "Footprint" "Capacitor_SMD:C_0805_2012Metric" (id 2) (at 143.3322 169.291 0)
       (effects (font (size 1.27 1.27)) hide)
     )
@@
     (property "Reference" "R105" (id 0) (at 154.305 155.0162 90))
     (property "Value" "R" (id 1) (at 154.305 157.3276 90))
-    (property "Footprint" "Resistor_SMD:R_1206_3216Metric" (id 2) (at 154.305 158.496 90)
+    (property "Footprint" "Resistor_SMD:R_0805_2012Metric" (id 2) (at 154.305 158.496 90)
       (effects (font (size 1.27 1.27)) hide)
     )
@@
       (effects (font (size 1.27 1.27)) (justify left))
     )
-    (property "Footprint" "Resistor_SMD:R_1206_3216Metric" (id 2) (at 94.742 156.464 90)
+    (property "Footprint" "Resistor_SMD:R_0805_2012Metric" (id 2) (at 94.742 156.464 90)
       (effects (font (size 1.27 1.27)) hide)
     )
@@
       (effects (font (size 1.27 1.27)) (justify left))
     )
-    (property "Footprint" "Capacitor_SMD:C_1206_3216Metric" (id 2) (at 97.4852 168.148 0)
+    (property "Footprint" "Capacitor_SMD:C_0805_2012Metric" (id 2) (at 97.4852 168.148 0)
       (effects (font (size 1.27 1.27)) hide)
     )

Commit message: new
Parts:
- removed D9: TVS 3,6V, Diode_SMD:D_1206_3216Metric, symbol lib_amplituner:1SMB5914BT3G
Changed lines of the file:
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@@
   (junction (at 162.56 80.01) (diameter 0) (color 0 0 0 0)
   )
-  (junction (at 127.635 170.688) (diameter 0) (color 0 0 0 0)
-  )
-  (junction (at 127.635 160.274) (diameter 0) (color 0 0 0 0)
-  )
   (junction (at 193.04 121.92) (diameter 0) (color 0 0 0 0)
   )
@@
     (stroke (width 0) (type default) (color 0 0 0 0))
   )
-  (wire (pts (xy 122.047 160.274) (xy 127.635 160.274))
+  (wire (pts (xy 122.047 160.274) (xy 142.367 160.274))
     (stroke (width 0) (type default) (color 0 0 0 0))
   )
@@
     (stroke (width 0) (type default) (color 0 0 0 0))
   )
-  (wire (pts (xy 127.635 160.274) (xy 142.367 160.274))
-    (stroke (width 0) (type default) (color 0 0 0 0))
-  )
   (wire (pts (xy 180.213 130.683) (xy 180.213 132.08))
     (stroke (width 0) (type default) (color 0 0 0 0))
@@
     (stroke (width 0) (type default) (color 0 0 0 0))
   )
-  (wire (pts (xy 114.427 170.688) (xy 127.635 170.688))
+  (wire (pts (xy 114.427 170.688) (xy 142.367 170.688))
     (stroke (width 0) (type default) (color 0 0 0 0))
   )
@@
     (stroke (width 0) (type default) (color 0 0 0 0))
   )
-  (wire (pts (xy 142.367 170.688) (xy 127.635 170.688))
-    (stroke (width 0) (type default) (color 0 0 0 0))
-  )
   (wire (pts (xy 158.115 160.274) (xy 159.512 160.274))
     (stroke (width 0) (type default) (color 0 0 0 0))
@@
   )
   (wire (pts (xy 111.76 80.01) (xy 118.11 80.01))
-    (stroke (width 0) (type default) (color 0 0 0 0))
-  )
-  (wire (pts (xy 127.635 160.274) (xy 127.635 160.528))
     (stroke (width 0) (type default) (color 0 0 0 0))
   )
@@
     (pin "1")
   )
-  (symbol (lib_id "lib_amplituner:1SMB5914BT3G") (at 127.635 165.608 90) (unit 1)
-    (in_bom yes) (on_board yes)
-    (property "Reference" "D9" (id 0) (at 129.667 164.4396 90)
-      (effects (font (size 1.27 1.27)) (justify right))
-    )
-    (property "Value" "TVS 3,6V" (id 1) (at 130.175 166.878 90)
-      (effects (font (size 1.27 1.27)) (justify right))
-    )
-    (property "Footprint" "Diode_SMD:D_1206_3216Metric" (id 2) (at 127.635 165.608 0)
-      (effects (font (size 1.27 1.27)) (justify left bottom) hide)
-    )
-    (property "Datasheet" "" (id 3) (at 127.635 165.608 0)
-      (effects (font (size 1.27 1.27)) (justify left bottom) hide)
-    )
-    (property "STANDARD" "IPC 7351B" (id 4) (at 127.635 165.608 0)
-      (effects (font (size 1.27 1.27)) (justify left bottom) hide)
-    )
-    (property "MANUFACTURER" "ON Semiconductor" (id 5) (at 127.635 165.608 0)
-      (effects (font (size 1.27 1.27)) (justify left bottom) hide)
-    )
-    (property "MAXIMUM_PACKAGE_HEIGHT" "2.47 mm" (id 6) (at 127.635 165.608 0)
-      (effects (font (size 1.27 1.27)) (justify left bottom) hide)
-    )
-    (property "PARTREV" "9" (id 7) (at 127.635 165.608 0)
-      (effects (font (size 1.27 1.27)) (justify left bottom) hide)
-    )
-    (pin "A")
-    (pin "C")
-  )
   (symbol (lib_id "Device:C") (at 96.52 164.338 0) (unit 1)
