File: Hardware/kicad/block diagram/block-sch/LM3886_scheet.kicad_sch (KiCad schematic)
At the start: 94 parts, among them U1 LM3886, U2 LM3886, U3 LM3886, U4 LM3886

Commit message: new
Parts:
- C11, C35, C36, C37, C38, C7, C8, C9: footprint Capacitor_THT:CP_Radial_D4.0mm_P2.00mm -> Capacitor_SMD:C_1206_3216Metric
- C13, C14, C25, C26, C47, C48, C49, C50: footprint Capacitor_THT:CP_Radial_D8.0mm_P2.50mm -> Capacitor_THT:CP_Radial_D12.5mm_P5.00mm
- C15, C17, C39, C40: footprint Capacitor_SMD:CP_Elec_4x3 -> Capacitor_THT:C_Radial_D8.0mm_H11.5mm_P3.50mm
- C16, C18, C41, C42: footprint Capacitor_THT:CP_Radial_D4.0mm_P2.00mm -> Capacitor_THT:C_Radial_D8.0mm_H11.5mm_P3.50mm
- C19, C20, C27, C28, C51, C52, C53, C54: footprint Capacitor_THT:CP_Radial_D8.0mm_P2.50mm -> Capacitor_THT:CP_Radial_D10.0mm_P5.00mm
- R10, R11, R20, R21, R22, R23, R24, R25, R6, R7, R8, R9: footprint Resistor_THT:R_Axial_DIN0309_L9.0mm_D3.2mm_P15.24mm_Horizontal -> Resistor_THT:R_Axial_DIN0204_L3.6mm_D1.6mm_P7.62mm_Horizontal
- R12, R14, R26, R27: footprint Resistor_THT:R_Axial_DIN0207_L6.3mm_D2.5mm_P7.62mm_Horizontal -> Resistor_THT:R_Axial_DIN0204_L3.6mm_D1.6mm_P7.62mm_Horizontal
Connections:
- net V+_2 is gone; now on net +36V: C45.1, C49.1, C53.1, C57.1, U4.1 (V+), U4.5 (V+)
- net V+_3 is gone; now on net +36V: C12.1, C14.1, C20.1, C24.1, U2.1 (V+), U2.5 (V+)
- net V+_4 is gone; now on net +36V: C22.1, C26.1, C28.1, C30.1, U1.1 (V+), U1.5 (V+)
- net V-_2 is gone; now on net -36V: C43.2, C47.2, C51.2, C55.2, R27.1, U4.4 (V-)
- net V-_3 is gone; now on net -36V: C10.2, C13.2, C19.2, C23.2, R14.1, U2.4 (V-)
- net V-_4 is gone; now on net -36V: C21.2, C25.2, C27.2, C29.2, R12.1, U1.4 (V-)
- net V+_1 renamed +36V
- net V-_1 renamed -36V

Commit message: new
Connections:
- net AUDIO_IN_LF is gone; now on net AUDIO_IN_RB: C31.2
- net AUDIO_IN_RB: no longer C3.2
- net AUDIO_IN_RF renamed Front_right_main
- new net Front_left_main: C3.2

Commit message: new
Connections:
- net SIG_GND renamed GNDA
Changed lines of the file:
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@@
     (effects (font (size 5.0038 5.0038) (thickness 1.0008) bold) (justify left bottom))
   )
-  (global_label "SIG_GND" (shape input) (at 172.72 87.63 180) (fields_autoplaced)
-    (effects (font (size 1.27 1.27)) (justify right))
-    (property "Intersheet References" "${INTERSHEET_REFS}" (id 0) (at 0 0 0)
-      (effects (font (size 1.27 1.27)) hide)
+  (global_label "GNDA" (shape input) (at 172.72 87.63 180) (fields_autoplaced)
+    (effects (font (size 1.27 1.27)) (justify right))
+    (property "Intersheet References" "${INTERSHEET_REFS}" (id 0) (at 165.4368 87.5506 0)
+      (effects (font (size 1.27 1.27)) (justify right) hide)
     )
   )
@@
     )
   )
-  (global_label "SIG_GND" (shape input) (at 58.42 86.36 180) (fields_autoplaced)
-    (effects (font (size 1.27 1.27)) (justify right))
-    (property "Intersheet References" "${INTERSHEET_REFS}" (id 0) (at 0 0 0)
-      (effects (font (size 1.27 1.27)) hide)
+  (global_label "GNDA" (shape input) (at 58.42 86.36 180) (fields_autoplaced)
+    (effects (font (size 1.27 1.27)) (justify right))
+    (property "Intersheet References" "${INTERSHEET_REFS}" (id 0) (at 51.1368 86.2806 0)
+      (effects (font (size 1.27 1.27)) (justify right) hide)
     )
   )
@@
     )
   )
-  (global_label "SIG_GND" (shape input) (at 147.32 53.34 180) (fields_autoplaced)
-    (effects (font (size 1.27 1.27)) (justify right))
-    (property "Intersheet References" "${INTERSHEET_REFS}" (id 0) (at 0 0 0)
-      (effects (font (size 1.27 1.27)) hide)
+  (global_label "GNDA" (shape input) (at 147.32 53.34 180) (fields_autoplaced)
+    (effects (font (size 1.27 1.27)) (justify right))
+    (property "Intersheet References" "${INTERSHEET_REFS}" (id 0) (at 140.0368 53.2606 0)
+      (effects (font (size 1.27 1.27)) (justify right) hide)
     )
   )
@@
     )
   )
-  (global_label "SIG_GND" (shape input) (at 33.02 52.07 180) (fields_autoplaced)
-    (effects (font (size 1.27 1.27)) (justify right))
-    (property "Intersheet References" "${INTERSHEET_REFS}" (id 0) (at 0 0 0)
-      (effects (font (size 1.27 1.27)) hide)
+  (global_label "GNDA" (shape input) (at 33.02 52.07 180) (fields_autoplaced)
+    (effects (font (size 1.27 1.27)) (justify right))
+    (property "Intersheet References" "${INTERSHEET_REFS}" (id 0) (at 25.7368 51.9906 0)
+      (effects (font (size 1.27 1.27)) (justify right) hide)
     )
   )
@@
     )
   )
-  (global_label "SIG_GND" (shape input) (at 175.26 156.21 180) (fields_autoplaced)
-    (effects (font (size 1.27 1.27)) (justify right))
-    (property "Intersheet References" "${INTERSHEET_REFS}" (id 0) (at 0 0 0)
-      (effects (font (size 1.27 1.27)) hide)
+  (global_label "GNDA" (shape input) (at 175.26 156.21 180) (fields_autoplaced)
+    (effects (font (size 1.27 1.27)) (justify right))
+    (property "Intersheet References" "${INTERSHEET_REFS}" (id 0) (at 167.9768 156.1306 0)
+      (effects (font (size 1.27 1.27)) (justify right) hide)
     )
   )
@@
     )
   )
-  (global_label "SIG_GND" (shape input) (at 53.34 189.23 180) (fields_autoplaced)
-    (effects (font (size 1.27 1.27)) (justify right))
-    (property "Intersheet References" "${INTERSHEET_REFS}" (id 0) (at 0 0 0)
-      (effects (font (size 1.27 1.27)) hide)
+  (global_label "GNDA" (shape input) (at 53.34 189.23 180) (fields_autoplaced)
+    (effects (font (size 1.27 1.27)) (justify right))
+    (property "Intersheet References" "${INTERSHEET_REFS}" (id 0) (at 46.0568 189.1506 0)
+      (effects (font (size 1.27 1.27)) (justify right) hide)
     )
   )
@@
     )
   )
-  (global_label "SIG_GND" (shape input) (at 27.94 154.94 180) (fields_autoplaced)
-    (effects (font (size 1.27 1.27)) (justify right))
-    (property "Intersheet References" "${INTERSHEET_REFS}" (id 0) (at 0 0 0)
-      (effects (font (size 1.27 1.27)) hide)
+  (global_label "GNDA" (shape input) (at 27.94 154.94 180) (fields_autoplaced)
+    (effects (font (size 1.27 1.27)) (justify right))
+    (property "Intersheet References" "${INTERSHEET_REFS}" (id 0) (at 20.6568 154.8606 0)
+      (effects (font (size 1.27 1.27)) (justify right) hide)
     )
   )
@@
     )
   )
-  (global_label "SIG_GND" (shape input) (at 149.86 121.92 180) (fields_autoplaced)
-    (effects (font (size 1.27 1.27)) (justify right))
-    (property "Intersheet References" "${INTERSHEET_REFS}" (id 0) (at 0 0 0)
-      (effects (font (size 1.27 1.27)) hide)
-    )
-  )
+  (global_label "GNDA" (shape input) (at 149.86 121.92 180) (fields_autoplaced)
+    (effects (font (size 1.27 1.27)) (justify right))
+    (property "Intersheet References" "${INTERSHEET_REFS}" (id 0) (at 142.5768 121.8406 0)
+      (effects (font (size 1.27 1.27)) (justify right) hide)
+    )
+  )
