File: Hardware/kicad/block diagram/block-sch/block-sch.kicad_sch (KiCad schematic)
At the start: 23 parts, among them K1 AZ850-x, Q1 BC817

Commit message: new
Parts:
- added C103, C104: 2200uF, Capacitor_THT:CP_Radial_D12.5mm_P5.00mm, symbol Device:CP_Small
- C1, C2: value 4700uF -> 2200uF
- D1: footprint Diode_THT:D_DO-201AE_P12.70mm_Horizontal -> Diode_THT:D_DO-35_SOD27_P7.62mm_Horizontal
- F2, F3: footprint (none) -> Fuse:Fuseholder_Cylinder-5x20mm_Schurter_0031_8201_Horizontal_Open
- K1: footprint Relay_THT:Relay_DPDT_FRT5 -> Relay_THT:Relay_DPDT_Fujitsu_FTR-F1C
Connections:
- net +15V: now also C103.1, C104.1
- net 12Vac: no longer D2.3, D2.4, TR1.11, TR1.12
- net GNDD: now also C103.2, C104.2
- net GNDPWR: no longer C1.2, C2.1, D3.1 (+), D4.2 (-)
- new net: D2.3, TR1.11
- new net: D2.4, TR1.12
- new net PWR_GND: C1.2, C2.1, D3.1 (+), D4.2 (-)
Other:
- moved on the sheet: F2, F3

Commit message: new
Parts:
- F1: footprint (none) -> Fuse:Fuse_1206_3216Metric
Connections:
- net 16V: no longer names the net of F1.2

Commit message: new
Connections:
- net STM32_Pin renamed Relay_POWER

Commit message: new
Other:
- added sheet Microphone (Microphones.kicad_sch)
- note added: "Microphones On board & external"
